File: digital_isolators.kicad_sch (KiCad schematic)
At the start: 9 parts, among them U4 ISO7760DBQ, U5 ISO7760DBQ, U6 ISO7760DBQ

Commit message: Started running traces
Parts:
- C_ISO_A1: renamed from C_ISO_A; footprint (none) -> Capacitor_SMD:C_0603_1608Metric
- C_ISO_B1: renamed from C_ISO_B; footprint (none) -> Capacitor_SMD:C_0603_1608Metric
- C_ISO_C1: renamed from C_ISO_C; footprint (none) -> Capacitor_SMD:C_0603_1608Metric
- C_ISO_D1: renamed from C_ISO_D; footprint (none) -> Capacitor_SMD:C_0603_1608Metric
- C_ISO_E1: renamed from C_ISO_E; footprint (none) -> Capacitor_SMD:C_0603_1608Metric
- C_ISO_F1: renamed from C_ISO_F; footprint (none) -> Capacitor_SMD:C_0603_1608Metric
Connections:
- net M2-BIN1 renamed M2_BIN1
Other:
- moved on the sheet: C_ISO_A1, C_ISO_B1, C_ISO_C1, C_ISO_D1, C_ISO_E1, C_ISO_F1, U4, U5, U6

Commit message: PCB tracing complete
Connections:
- net GND_ISO: now also U6.3 (INB), U6.4 (INC), U6.5 (IND); no longer U5.5 (IND), U5.6 (INE), U5.7 (INF)
- net ISO_M2_CLOSE: now also U4.6 (INE); no longer U4.5 (IND)
- net ISO_M2_OPEN: now also U4.5 (IND); no longer U4.4 (INC)
- net ISO_M3_CLOSE: now also U5.3 (INB); no longer U4.7 (INF)
- net ISO_M3_OPEN: now also U5.4 (INC); no longer U4.6 (INE)
- net ISO_M4_CLOSE: now also U5.6 (INE); no longer U5.3 (INB)
- net ISO_M4_OPEN: now also U5.5 (IND); no longer U5.2 (INA)
- net ISO_PWM_M1: now also U4.4 (INC); no longer U6.2 (INA)
- net ISO_PWM_M2: now also U4.7 (INF); no longer U6.3 (INB)
- net ISO_PWM_M3: now also U5.2 (INA); no longer U6.4 (INC)
- net ISO_PWM_M4: now also U5.7 (INF); no longer U6.5 (IND)
- net ISO_STBY: now also U6.2 (INA); no longer U5.4 (INC)
- net M2_BIN1: now also U4.12 (OUTD); no longer U4.13 (OUTC)
- net M2_BIN2: now also U4.11 (OUTE); no longer U4.12 (OUTD)
- net M3_AIN1: now also U5.13 (OUTC); no longer U4.11 (OUTE)
- net M3_AIN2: now also U5.14 (OUTB); no longer U4.10 (OUTF)
- net M4_BIN1: now also U5.12 (OUTD); no longer U5.15 (OUTA)
- net M4_BIN2: now also U5.11 (OUTE); no longer U5.14 (OUTB)
- net PWM_M1: now also U4.13 (OUTC); no longer U6.15 (OUTA)
- net PWM_M2: now also U4.10 (OUTF); no longer U6.14 (OUTB)
- net PWM_M3: now also U5.15 (OUTA); no longer U6.13 (OUTC)
- net PWM_M4: now also U5.10 (OUTF); no longer U6.12 (OUTD)
- net STBY: now also U6.15 (OUTA); no longer U5.13 (OUTC)

Commit message: BOM work
Parts:
- C_ISO_A1, C_ISO_B1, C_ISO_C1, C_ISO_D1, C_ISO_E1, C_ISO_F1: LCSC (none) -> C1590
- U4, U5, U6: LCSC (none) -> C2868628
Changed lines of the file:
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@@
 		(dnp no)
 		(fields_autoplaced yes)
-		(property "Reference" "#PWR057"
+		(property "Reference" "#PWR043"
 			(at 214.63 60.96 0)
 			(effects
@@
 			(project "barn-blinds-controller"
 				(path "/aa90962a-81b9-423d-8acd-c4e83fa798bb/5abc6c0d-fca0-406e-b928-fa5bf81b9020"
-					(reference "#PWR057")
+					(reference "#PWR043")
 					(unit 1)
 				)
@@
 			)
 		)
+		(property "LCSC" "C2868628"
+			(at 219.71 87.63 0)
+			(effects
+				(font
+					(size 1.27 1.27)
+				)
+				(hide yes)
+			)
+		)
 		(pin "6"
 		)
@@
 		(dnp no)
 		(fields_autoplaced yes)
-		(property "Reference" "#PWR055"
+		(property "Reference" "#PWR026"
 			(at 78.74 58.42 0)
 			(effects
@@
 			(project "barn-blinds-controller"
 				(path "/aa90962a-81b9-423d-8acd-c4e83fa798bb/5abc6c0d-fca0-406e-b928-fa5bf81b9020"
-					(reference "#PWR055")
+					(reference "#PWR026")
 					(unit 1)
 				)
@@
 		(dnp no)
 		(fields_autoplaced yes)
-		(property "Reference" "#PWR061"
+		(property "Reference" "#PWR028"
 			(at 88.9 57.15 0)
 			(effects
@@
 			(project "barn-blinds-controller"
 				(path "/aa90962a-81b9-423d-8acd-c4e83fa798bb/5abc6c0d-fca0-406e-b928-fa5bf81b9020"
-					(reference "#PWR061")
+					(reference "#PWR028")
 					(unit 1)
 				)
@@
 		(dnp no)
 		(fields_autoplaced yes)
-		(property "Reference" "#PWR072"
+		(property "Reference" "#PWR030"
 			(at 102.87 59.69 0)
 			(effects
@@
 			(project "barn-blinds-controller"
 				(path "/aa90962a-81b9-423d-8acd-c4e83fa798bb/5abc6c0d-fca0-406e-b928-fa5bf81b9020"
-					(reference "#PWR072")
+					(reference "#PWR030")
 					(unit 1)
 				)
@@
 		(dnp no)
 		(fields_autoplaced yes)
-		(property "Reference" "#PWR076"
+		(property "Reference" "#PWR041"
 			(at 203.2 90.17 0)
 			(effects
@@
 			(project "barn-blinds-controller"
 				(path "/aa90962a-81b9-423d-8acd-c4e83fa798bb/5abc6c0d-fca0-406e-b928-fa5bf81b9020"
-					(reference "#PWR076")
+					(reference "#PWR041")
 					(unit 1)
 				)
@@
 		(dnp no)
 		(fields_autoplaced yes)
-		(property "Reference" "#PWR088"
+		(property "Reference" "#PWR038"
 			(at 203.2 82.55 0)
 			(effects
@@
 			(project "barn-blinds-controller"
 				(path "/aa90962a-81b9-423d-8acd-c4e83fa798bb/5abc6c0d-fca0-406e-b928-fa5bf81b9020"
-					(reference "#PWR088")
+					(reference "#PWR038")
 					(unit 1)
 				)
@@
 		(dnp no)
 		(fields_autoplaced yes)
-		(property "Reference" "#PWR064"
+		(property "Reference" "#PWR029"
 			(at 88.9 105.41 0)
 			(effects
@@
 			(project "barn-blinds-controller"
 				(path "/aa90962a-81b9-423d-8acd-c4e83fa798bb/5abc6c0d-fca0-406e-b928-fa5bf81b9020"
-					(reference "#PWR064")
+					(reference "#PWR029")
 					(unit 1)
 				)
@@
 			)
 		)
+		(property "LCSC" "C2868628"
+			(at 83.82 83.82 0)
+			(effects
+				(font
+					(size 1.27 1.27)
+				)
+				(hide yes)
+			)
+		)
 		(pin "6"
 		)
@@
 		(dnp no)
 		(fields_autoplaced yes)
-		(property "Reference" "#PWR071"
+		(property "Reference" "#PWR036"
 			(at 171.45 60.96 0)
 			(effects
@@
 			(project "barn-blinds-controller"
 				(path "/aa90962a-81b9-423d-8acd-c4e83fa798bb/5abc6c0d-fca0-406e-b928-fa5bf81b9020"
-					(reference "#PWR071")
+					(reference "#PWR036")
 					(unit 1)
 				)
@@
 		(dnp no)
 		(fields_autoplaced yes)
-		(property "Reference" "#PWR077"
+		(property "Reference" "#PWR042"
 			(at 203.2 92.71 0)
 			(effects
@@
 			(project "barn-blinds-controller"
 				(path "/aa90962a-81b9-423d-8acd-c4e83fa798bb/5abc6c0d-fca0-406e-b928-fa5bf81b9020"
-					(reference "#PWR077")
+					(reference "#PWR042")
 					(unit 1)
 				)
@@
 		(dnp no)
 		(fields_autoplaced yes)
-		(property "Reference" "#PWR066"
+		(property "Reference" "#PWR046"
 			(at 224.79 109.22 0)
 			(effects
@@
 			(project "barn-blinds-controller"
 				(path "/aa90962a-81b9-423d-8acd-c4e83fa798bb/5abc6c0d-fca0-406e-b928-fa5bf81b9020"
-					(reference "#PWR066")
+					(reference "#PWR046")
 					(unit 1)
 				)
@@
 		(dnp no)
 		(fields_autoplaced yes)
-		(property "Reference" "#PWR068"
+		(property "Reference" "#PWR031"
 			(at 138.43 68.58 0)
 			(effects
@@
 			(project "barn-blinds-controller"
 				(path "/aa90962a-81b9-423d-8acd-c4e83fa798bb/5abc6c0d-fca0-406e-b928-fa5bf81b9020"
-					(reference "#PWR068")
+					(reference "#PWR031")
 					(unit 1)
 				)
@@
 		(dnp no)
 		(fields_autoplaced yes)
-		(property "Reference" "#PWR069"
+		(property "Reference" "#PWR037"
 			(at 205.74 71.12 0)
 			(effects
@@
 			(project "barn-blinds-controller"
 				(path "/aa90962a-81b9-423d-8acd-c4e83fa798bb/5abc6c0d-fca0-406e-b928-fa5bf81b9020"
-					(reference "#PWR069")
+					(reference "#PWR037")
 					(unit 1)
 				)
@@
 		(dnp no)
 		(fields_autoplaced yes)
-		(property "Reference" "#PWR059"
+		(property "Reference" "#PWR044"
 			(at 214.63 109.22 0)
 			(effects
@@
 			(project "barn-blinds-controller"
 				(path "/aa90962a-81b9-423d-8acd-c4e83fa798bb/5abc6c0d-fca0-406e-b928-fa5bf81b9020"
-					(reference "#PWR059")
+					(reference "#PWR044")
 					(unit 1)
 				)
@@
 			)
 		)
+		(property "LCSC" "C2868628"
+			(at 152.4 85.09 0)
+			(effects
+				(font
+					(size 1.27 1.27)
+				)
+				(hide yes)
+			)
+		)
 		(pin "6"
 		)
@@
 		(dnp no)
 		(fields_autoplaced yes)
-		(property "Reference" "#PWR060"
+		(property "Reference" "#PWR027"
 			(at 78.74 105.41 0)
 			(effects
@@
 			(project "barn-blinds-controller"
 				(path "/aa90962a-81b9-423d-8acd-c4e83fa798bb/5abc6c0d-fca0-406e-b928-fa5bf81b9020"
-					(reference "#PWR060")
+					(reference "#PWR027")
 					(unit 1)
 				)
@@
 		(dnp no)
 		(fields_autoplaced yes)
-		(property "Reference" "#PWR058"
+		(property "Reference" "#PWR033"
 			(at 147.32 106.68 0)
 			(effects
@@
 			(project "barn-blinds-controller"
 				(path "/aa90962a-81b9-423d-8acd-c4e83fa798bb/5abc6c0d-fca0-406e-b928-fa5bf81b9020"
-					(reference "#PWR058")
+					(reference "#PWR033")
 					(unit 1)
 				)
@@
 		(dnp no)
 		(fields_autoplaced yes)
-		(property "Reference" "#PWR056"
+		(property "Reference" "#PWR032"
 			(at 147.32 59.69 0)
 			(effects
@@
 			(project "barn-blinds-controller"
 				(path "/aa90962a-81b9-423d-8acd-c4e83fa798bb/5abc6c0d-fca0-406e-b928-fa5bf81b9020"
-					(reference "#PWR056")
+					(reference "#PWR032")
 					(unit 1)
 				)
@@
 		(dnp no)
 		(fields_autoplaced yes)
-		(property "Reference" "#PWR062"
+		(property "Reference" "#PWR034"
 			(at 157.48 57.15 0)
 			(effects
@@
 			(project "barn-blinds-controller"
 				(path "/aa90962a-81b9-423d-8acd-c4e83fa798bb/5abc6c0d-fca0-406e-b928-fa5bf81b9020"
-					(reference "#PWR062")
+					(reference "#PWR034")
 					(unit 1)
 				)
@@
 		(dnp no)
 		(fields_autoplaced yes)
-		(property "Reference" "#PWR073"
+		(property "Reference" "#PWR039"
 			(at 203.2 85.09 0)
 			(effects
@@
 			(project "barn-blinds-controller"
 				(path "/aa90962a-81b9-423d-8acd-c4e83fa798bb/5abc6c0d-fca0-406e-b928-fa5bf81b9020"
-					(reference "#PWR073")
+					(reference "#PWR039")
 					(unit 1)
 				)
@@
 			)
 		)
+		(property "LCSC" "C1590"
+			(at 73.66 59.69 90)
+			(effects
+				(font
+					(size 1.27 1.27)
+				)
+				(hide yes)
+			)
+		)
 		(pin "1"
 		)
@@
 			)
 		)
+		(property "LCSC" "C1590"
+			(at 229.87 63.5 90)
+			(effects
+				(font
+					(size 1.27 1.27)
+				)
+				(hide yes)
+			)
+		)
 		(pin "1"
 		)
@@
 		(dnp no)
 		(fields_autoplaced yes)
-		(property "Reference" "#PWR070"
+		(property "Reference" "#PWR047"
 			(at 238.76 63.5 0)
 			(effects
@@
 			(project "barn-blinds-controller"
 				(path "/aa90962a-81b9-423d-8acd-c4e83fa798bb/5abc6c0d-fca0-406e-b928-fa5bf81b9020"
-					(reference "#PWR070")
+					(reference "#PWR047")
 					(unit 1)
 				)
@@
 			)
 		)
+		(property "LCSC" "C1590"
+			(at 162.56 60.96 90)
+			(effects
+				(font
+					(size 1.27 1.27)
+				)
+				(hide yes)
+			)
+		)
 		(pin "1"
 		)
@@
 			)
 		)
+		(property "LCSC" "C1590"
+			(at 142.24 62.23 90)
+			(effects
+				(font
+					(size 1.27 1.27)
+				)
+				(hide yes)
+			)
+		)
 		(pin "1"
 		)
@@
 			)
 		)
+		(property "LCSC" "C1590"
+			(at 93.98 59.69 90)
+			(effects
+				(font
+					(size 1.27 1.27)
+				)
+				(hide yes)
+			)
+		)
 		(pin "1"
 		)
@@
 		(dnp no)
 		(fields_autoplaced yes)
-		(property "Reference" "#PWR074"
+		(property "Reference" "#PWR040"
 			(at 203.2 87.63 0)
 			(effects
@@
 			(project "barn-blinds-controller"
 				(path "/aa90962a-81b9-423d-8acd-c4e83fa798bb/5abc6c0d-fca0-406e-b928-fa5bf81b9020"
-					(reference "#PWR074")
+					(reference "#PWR040")
 					(unit 1)
 				)
@@
 		(dnp no)
 		(fields_autoplaced yes)
-		(property "Reference" "#PWR065"
+		(property "Reference" "#PWR035"
 			(at 157.48 106.68 0)
 			(effects
@@
 			(project "barn-blinds-controller"
 				(path "/aa90962a-81b9-423d-8acd-c4e83fa798bb/5abc6c0d-fca0-406e-b928-fa5bf81b9020"
-					(reference "#PWR065")
+					(reference "#PWR035")
 					(unit 1)
 				)
@@
 		(dnp no)
 		(fields_autoplaced yes)
-		(property "Reference" "#PWR063"
+		(property "Reference" "#PWR045"
 			(at 224.79 58.42 0)
 			(effects
@@
 			(project "barn-blinds-controller"
 				(path "/aa90962a-81b9-423d-8acd-c4e83fa798bb/5abc6c0d-fca0-406e-b928-fa5bf81b9020"
-					(reference "#PWR063")
+					(reference "#PWR045")
 					(unit 1)
 				)
@@
 		(dnp no)
 		(fields_autoplaced yes)
-		(property "Reference" "#PWR067"
+		(property "Reference" "#PWR025"
 			(at 68.58 66.04 0)
 			(effects
@@
 			(project "barn-blinds-controller"
 				(path "/aa90962a-81b9-423d-8acd-c4e83fa798bb/5abc6c0d-fca0-406e-b928-fa5bf81b9020"
-					(reference "#PWR067")
+					(reference "#PWR025")
 					(unit 1)
 				)
@@
 			(effects
 				(font
+					(size 1.27 1.27)
+				)
+				(hide yes)
+			)
+		)
+		(property "LCSC" "C1590"
+			(at 209.55 64.77 90)
+			(effects
+				(font

Commit message: Refactored board to use larger vias and route better paths.
Connections:
- net GND_ISO: now also U5.2 (INA), U5.3 (INB), U5.4 (INC), U5.5 (IND), U5.6 (INE); no longer U6.3 (INB), U6.4 (INC), U6.5 (IND), U6.6 (INE), U6.7 (INF)
- net ISO_M1_CLOSE: now also U4.6 (INE); no longer U4.3 (INB)
- net ISO_M1_OPEN: now also U4.5 (IND); no longer U4.2 (INA)
- net ISO_M2_CLOSE: now also U4.3 (INB); no longer U4.6 (INE)
- net ISO_M2_OPEN: now also U4.4 (INC); no longer U4.5 (IND)
- net ISO_M3_CLOSE: now also U6.6 (INE); no longer U5.3 (INB)
- net ISO_M3_OPEN: now also U6.5 (IND); no longer U5.4 (INC)
- net ISO_M4_CLOSE: now also U6.2 (INA); no longer U5.6 (INE)
- net ISO_M4_OPEN: now also U6.3 (INB); no longer U5.5 (IND)
- net ISO_PWM_M1: now also U4.7 (INF); no longer U4.4 (INC)
- net ISO_PWM_M2: now also U4.2 (INA); no longer U4.7 (INF)
- net ISO_PWM_M3: now also U6.7 (INF); no longer U5.2 (INA)
- net ISO_STBY: now also U6.4 (INC); no longer U6.2 (INA)
- net M1_AIN1: now also U4.12 (OUTD); no longer U4.15 (OUTA)
- net M1_AIN2: now also U4.11 (OUTE); no longer U4.14 (OUTB)
- net M2_BIN1: now also U4.13 (OUTC); no longer U4.12 (OUTD)
- net M2_BIN2: now also U4.14 (OUTB); no longer U4.11 (OUTE)
- net M3_AIN1: now also U6.12 (OUTD); no longer U5.13 (OUTC)
- net M3_AIN2: now also U6.11 (OUTE); no longer U5.14 (OUTB)
- net M4_BIN1: now also U6.14 (OUTB); no longer U5.12 (OUTD)
- net M4_BIN2: now also U6.15 (OUTA); no longer U5.11 (OUTE)
- net PWM_M1: now also U4.10 (OUTF); no longer U4.13 (OUTC)
- net PWM_M2: now also U4.15 (OUTA); no longer U4.10 (OUTF)
- net PWM_M3: now also U6.10 (OUTF); no longer U5.15 (OUTA)
- net STBY: now also U6.13 (OUTC); no longer U6.15 (OUTA)
