File: digital_isolators.kicad_sch (KiCad schematic)
At the start: 9 parts, among them U4 ISO7760DBQ, U5 ISO7760DBQ, U6 ISO7760DBQ

Commit message: Updating routing with new terminal block
Connections:
- net ISO_M1_CLOSE renamed ISO_SH4_CLOSE
- net ISO_M1_OPEN renamed ISO_SH4_OPEN
- net ISO_M2_CLOSE renamed ISO_SH3_CLOSED
- net ISO_M2_OPEN renamed ISO_SH3_OPEN
- net ISO_M3_CLOSE renamed ISO_SH2_CLOSED
- net ISO_M3_OPEN renamed ISO_SH2_OPEN
- net ISO_M4_CLOSE renamed ISO_SH1_CLOSED
- net ISO_M4_OPEN renamed ISO_SH1_OPEN
- net ISO_PWM_M1 renamed ISO_SH4_PWM
- net ISO_PWM_M2 renamed ISO_SH3_PWM
- net ISO_PWM_M3 renamed ISO_SH2_PWM
- net ISO_PWM_M4 renamed ISO_SH1_PWM
- net M1_AIN1 renamed SH4_IN1
- net M1_AIN2 renamed SH4_IN2
- net M2_BIN1 renamed SH3_IN1
- net M2_BIN2 renamed SH3_IN2
- net M3_AIN1 renamed SH2_IN1
- net M3_AIN2 renamed SH2_IN2
- net M4_BIN1 renamed SH1_IN1
- net M4_BIN2 renamed SH1_IN2
- net PWM_M1 renamed SH4_PWM
- net PWM_M2 renamed SH3_PWM
- net PWM_M3 renamed SH2_PWM
- net PWM_M4 renamed SH1_PWM

Commit message: Added RTS/DTS programing via UART circuitry, added LED control circuitry.
Parts:
- added R17: 10K, Resistor_SMD:R_0603_1608Metric, symbol Device:R
Connections:
- net +3.3V_ISO: now also R17.1
- net GND_ISO: no longer U5.2 (INA)
- net LED_D5_SW: now reaches U5.15 (OUTA)
- new net LED_D5_CTRL: R17.2, U5.2 (INA)
- no-connect marks 5 -> 4
Changed lines of the file:
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@@
 	)
 	(no_connect
-		(at 162.56 77.47)
-	)
-	(no_connect
 		(at 162.56 85.09)
 	)
@@
 	(wire
 		(pts
+			(xy 109.22 100.33) (xy 109.22 106.68)
+		)
+		(stroke
+			(width 0)
+			(type default)
+		)
+	)
+	(wire
+		(pts
 			(xy 88.9 53.34) (xy 88.9 59.69)
 		)
@@
 		)
 	)
+	(global_label "LED_D5_SW"
+		(shape input)
+		(at 162.56 77.47 0)
+		(fields_autoplaced yes)
+		(effects
+			(font
+				(size 1.27 1.27)
+			)
+			(justify left)
+		)
+		(property "Intersheetrefs" "${INTERSHEET_REFS}"
+			(at 172.7418 77.47 0)
+			(hide yes)
+			(show_name no)
+			(do_not_autoplace no)
+			(effects
+				(font
+					(size 1.27 1.27)
+				)
+				(justify left)
+			)
+		)
+	)
 	(global_label "SH1_IN2"
 		(shape input)
@@
 		)
 	)
+	(global_label "LED_D5_CTRL"
+		(shape input)
+		(at 142.24 77.47 180)
+		(fields_autoplaced yes)
+		(effects
+			(font
+				(size 1.27 1.27)
+			)
+			(justify right)
+		)
+		(property "Intersheetrefs" "${INTERSHEET_REFS}"
+			(at 132.08 77.47 0)
+			(hide yes)
+			(show_name no)
+			(do_not_autoplace no)
+			(effects
+				(font
+					(size 1.27 1.27)
+				)
+				(justify left)
+			)
+		)
+	)
 	(global_label "STBY"
 		(shape bidirectional)
@@
 		)
 	)
+	(global_label "LED_D5_CTRL"
+		(shape input)
+		(at 109.22 114.3 270)
+		(fields_autoplaced yes)
+		(effects
+			(font
+				(size 1.27 1.27)
+			)
+			(justify right)
+		)
+		(property "Intersheetrefs" "${INTERSHEET_REFS}"
+			(at 109.22 129.6827 90)
+			(hide yes)
+			(show_name no)
+			(do_not_autoplace no)
+			(effects
+				(font
+					(size 1.27 1.27)
+				)
+				(justify right)
+			)
+		)
+	)
 	(global_label "ISO_SH2_PWM"
 		(shape input)
@@
 	)
 	(symbol
+		(lib_id "Device:R")
+		(at 109.22 110.49 0)
+		(unit 1)
+		(body_style 1)
+		(exclude_from_sim no)
+		(in_bom yes)
+		(on_board yes)
+		(in_pos_files yes)
+		(dnp no)
+		(fields_autoplaced yes)
+		(property "Reference" "R17"
+			(at 111.76 109.22 0)
+			(show_name no)
+			(do_not_autoplace no)
+			(effects
+				(font
+					(size 1.27 1.27)
+				)
+				(justify left)
+			)
+		)
+		(property "Value" "10K"
+			(at 111.76 111.76 0)
+			(show_name no)
+			(do_not_autoplace no)
+			(effects
+				(font
+					(size 1.27 1.27)
+				)
+				(justify left)
+			)
+		)
+		(property "Footprint" "Resistor_SMD:R_0603_1608Metric"
+			(at 107.442 110.49 90)
+			(hide yes)
+			(show_name no)
+			(do_not_autoplace no)
+			(effects
+				(font
+					(size 1.27 1.27)
+				)
+			)
+		)
+		(property "Datasheet" ""
+			(at 109.22 110.49 0)
+			(hide yes)
+			(show_name no)
+			(do_not_autoplace no)
+			(effects
+				(font
+					(size 1.27 1.27)
+				)
+			)
+		)
+		(property "Description" "Resistor"
+			(at 109.22 110.49 0)
+			(hide yes)
+			(show_name no)
+			(do_not_autoplace no)
+			(effects
+				(font
+					(size 1.27 1.27)
+				)
+			)
+		)
+		(property "LCSC" "C25804"
+			(at 109.22 110.49 0)
+			(hide yes)
+			(show_name no)
+			(do_not_autoplace no)
+			(effects
+				(font
+					(size 1.27 1.27)
+				)
+			)
+		)
+		(pin "1"
+		)
+		(pin "2"
+		)
+		(instances
+			(project "barn-blinds-controller"
+				(path "/aa90962a-81b9-423d-8acd-c4e83fa798bb/5abc6c0d-fca0-406e-b928-fa5bf81b9020"
+					(reference "R17")
+					(unit 1)
+				)
+			)
+		)
+	)
+	(symbol
 		(lib_id "Device:C")
 		(at 73.66 59.69 90)
@@
 	(symbol
 		(lib_id "power:GND")
-		(at 142.24 77.47 270)
+		(at 142.24 87.63 270)
 		(unit 1)
 		(body_style 1)
@@
 		(dnp no)
 		(fields_autoplaced yes)
-		(property "Reference" "#PWR032"
-			(at 135.89 77.47 0)
+		(property "Reference" "#PWR036"
+			(at 135.89 87.63 0)
 			(hide yes)
 			(show_name no)
@@
 		)
 		(property "Value" "GND_ISO"
-			(at 138.43 77.4699 90)
+			(at 138.43 87.6299 90)
 			(show_name no)
 			(do_not_autoplace no)
@@
 		)
 		(property "Footprint" ""
-			(at 142.24 77.47 0)
+			(at 142.24 87.63 0)
 			(hide yes)
 			(show_name no)
@@
 		)
 		(property "Datasheet" ""
-			(at 142.24 77.47 0)
+			(at 142.24 87.63 0)
 			(hide yes)
 			(show_name no)
@@
 		)
 		(property "Description" "Power symbol creates a global label with name \"GND\" , ground"
-			(at 142.24 77.47 0)
+			(at 142.24 87.63 0)
 			(hide yes)
 			(show_name no)
@@
 			(project "barn-blinds-controller"
 				(path "/aa90962a-81b9-423d-8acd-c4e83fa798bb/5abc6c0d-fca0-406e-b928-fa5bf81b9020"
-					(reference "#PWR032")
+					(reference "#PWR036")
 					(unit 1)
 				)
@@
 	)
 	(symbol
-		(lib_id "power:GND")
-		(at 142.24 87.63 270)
+		(lib_id "Device:C")
+		(at 93.98 59.69 90)
 		(unit 1)
 		(body_style 1)
@@
 		(dnp no)
 		(fields_autoplaced yes)
-		(property "Reference" "#PWR036"
-			(at 135.89 87.63 0)
-			(hide yes)
+		(property "Reference" "C_ISO_B1"
+			(at 93.98 52.07 90)
 			(show_name no)
 			(do_not_autoplace no)
@@
 			)
 		)
-		(property "Value" "GND_ISO"
-			(at 138.43 87.6299 90)
+		(property "Value" "0.1uF"
+			(at 93.98 54.61 90)
 			(show_name no)
 			(do_not_autoplace no)
@@
 					(size 1.27 1.27)
 				)
-				(justify right)
 			)
 		)
-		(property "Footprint" ""
-			(at 142.24 87.63 0)
+		(property "Footprint" "Capacitor_SMD:C_0603_1608Metric"
+			(at 97.79 58.7248 0)
 			(hide yes)
 			(show_name no)
@@
 		)
 		(property "Datasheet" ""
-			(at 142.24 87.63 0)
+			(at 93.98 59.69 0)
 			(hide yes)
 			(show_name no)
@@
 			)
 		)
-		(property "Description" "Power symbol creates a global label with name \"GND\" , ground"
-			(at 142.24 87.63 0)
+		(property "Description" "Unpolarized capacitor"
+			(at 93.98 59.69 0)
+			(hide yes)
+			(show_name no)
+			(do_not_autoplace no)
+			(effects
+				(font
+					(size 1.27 1.27)
+				)
+			)
+		)
+		(property "LCSC" "C1590"
+			(at 93.98 59.69 90)
 			(hide yes)
 			(show_name no)
@@
 		(pin "1"
 		)
+		(pin "2"
+		)
 		(instances
 			(project "barn-blinds-controller"
 				(path "/aa90962a-81b9-423d-8acd-c4e83fa798bb/5abc6c0d-fca0-406e-b928-fa5bf81b9020"
-					(reference "#PWR036")
+					(reference "C_ISO_B1")
 					(unit 1)
 				)
@@
 	)
 	(symbol
-		(lib_id "Device:C")
-		(at 93.98 59.69 90)
+		(lib_id "power:GND")
+		(at 157.48 100.33 0)
 		(unit 1)
 		(body_style 1)
@@
 		(dnp no)
 		(fields_autoplaced yes)
-		(property "Reference" "C_ISO_B1"
-			(at 93.98 52.07 90)
+		(property "Reference" "#PWR040"
+			(at 157.48 106.68 0)
+			(hide yes)
 			(show_name no)
 			(do_not_autoplace no)
@@
 			)
 		)
-		(property "Value" "0.1uF"
-			(at 93.98 54.61 90)
+		(property "Value" "GND_MOTOR"
+			(at 157.48 105.41 0)
 			(show_name no)
 			(do_not_autoplace no)
@@
 			)
 		)
-		(property "Footprint" "Capacitor_SMD:C_0603_1608Metric"
-			(at 97.79 58.7248 0)
+		(property "Footprint" ""
+			(at 157.48 100.33 0)
 			(hide yes)
 			(show_name no)
@@
 		)
 		(property "Datasheet" ""
-			(at 93.98 59.69 0)
-			(hide yes)
-			(show_name no)
-			(do_not_autoplace no)
-			(effects
-				(font
-					(size 1.27 1.27)
-				)
-			)
-		)
-		(property "Description" "Unpolarized capacitor"
-			(at 93.98 59.69 0)
+			(at 157.48 100.33 0)
 			(hide yes)
 			(show_name no)
@@
 			)
 		)
-		(property "LCSC" "C1590"
-			(at 93.98 59.69 90)
+		(property "Description" "Power symbol creates a global label with name \"GND\" , ground"
+			(at 157.48 100.33 0)
 			(hide yes)
 			(show_name no)
@@
 		(pin "1"
 		)
-		(pin "2"
-		)
 		(instances
 			(project "barn-blinds-controller"
 				(path "/aa90962a-81b9-423d-8acd-c4e83fa798bb/5abc6c0d-fca0-406e-b928-fa5bf81b9020"
-					(reference "C_ISO_B1")
+					(reference "#PWR040")
 					(unit 1)
 				)
@@
 	)
 	(symbol
-		(lib_id "power:GND")
-		(at 157.48 100.33 0)
+		(lib_id "power:+3.3V")
+		(at 109.22 100.33 0)
 		(unit 1)
 		(body_style 1)
@@
 		(dnp no)
 		(fields_autoplaced yes)
-		(property "Reference" "#PWR040"
-			(at 157.48 106.68 0)
+		(property "Reference" "#PWR0120"
+			(at 109.22 96.33 0)
 			(hide yes)
 			(show_name no)
@@
 			)
 		)
-		(property "Value" "GND_MOTOR"
-			(at 157.48 105.41 0)
+		(property "Value" "+3.3V_ISO"
+			(at 109.22 95.25 0)
 			(show_name no)
 			(do_not_autoplace no)
@@
 		)
 		(property "Footprint" ""
-			(at 157.48 100.33 0)
+			(at 109.22 100.33 0)
 			(hide yes)
 			(show_name no)
@@
 		)
 		(property "Datasheet" ""
-			(at 157.48 100.33 0)
+			(at 109.22 100.33 0)
 			(hide yes)
 			(show_name no)
@@
 			)
 		)
-		(property "Description" "Power symbol creates a global label with name \"GND\" , ground"
-			(at 157.48 100.33 0)
+		(property "Description" "Power symbol creates a global label with name \"+3V3\""
+			(at 109.22 100.33 0)
 			(hide yes)
 			(show_name no)
@@
 			(project "barn-blinds-controller"
 				(path "/aa90962a-81b9-423d-8acd-c4e83fa798bb/5abc6c0d-fca0-406e-b928-fa5bf81b9020"
-					(reference "#PWR040")
+					(reference "#PWR0120")
 					(unit 1)
 				)

Commit message: Update annotations, fixed font sizes.
Parts:
- renumbered C_ISO_A1 to C22, C_ISO_B1 to C23, C_ISO_C1 to C24, C_ISO_D1 to C25, C_ISO_E1 to C26, C_ISO_F1 to C27
