File: esp32-s3.kicad_sch (KiCad schematic)
At the start: 9 parts, among them SW1 BOOT, SW2 RESET, U1 ESP32-S3-WROOM-1

Commit message: Started running traces
Parts:
- C33: footprint (none) -> Capacitor_SMD:C_0805_2012Metric
- C34: footprint (none) -> Capacitor_SMD:C_0603_1608Metric
- R2: value R -> 10K; footprint (none) -> Resistor_SMD:R_0603_1608Metric
- R_BOOT1: renamed from R_BOOT; footprint (none) -> Resistor_SMD:R_0603_1608Metric
- R_LED1: renamed from R_LED; value 150R -> 470R; footprint (none) -> Resistor_SMD:R_0603_1608Metric
- SW1, SW2: footprint (none) -> barn_shade_controller:SW-SMD_4P-L3.5-W3.0-P1.50-LS4.7; symbol Switch:SW_Push -> Switch:SW_Push_Open_Dual
Connections:
- net GND_ISO: now also SW1.4, SW2.3
- net at R2.2, SW2.2, U1.3 (EN): now also SW2.4
- net at R_BOOT1.1, SW1.1, U1.27 (GPIO0/BOOT): now also SW1.3

Commit message: Started running traces
Connections:
- net ISO_M2_CLOSE: now also U1.36 (U0RXD/GPIO44/CLK_OUT2); no longer U1.4 (GPIO4/TOUCH4/ADC1_CH3)
- net ISO_M2_OPEN: now also U1.37 (U0TXD/GPIO43/CLK_OUT1); no longer U1.15 (GPIO3/TOUCH3/ADC1_CH2)
- net ISO_M3_CLOSE: now also U1.34 (MTDI/GPIO41/CLK_OUT1); no longer U1.6 (GPIO6/TOUCH6/ADC1_CH5)
- net ISO_M3_OPEN: now also U1.35 (MTMS/GPIO42); no longer U1.5 (GPIO5/TOUCH5/ADC1_CH4)
- net ISO_M4_CLOSE: now also U1.32 (MTCK/GPIO39/CLK_OUT3/SUBSPICS1); no longer U1.12 (GPIO8/TOUCH8/ADC1_CH7/SUBSPICS1)
- net ISO_M4_OPEN: now also U1.33 (MTDO/GPIO40/CLK_OUT2); no longer U1.7 (GPIO7/TOUCH7/ADC1_CH6)
- net ISO_PWM_M1: now also U1.30 (SPIDQS/GPIO37/FSPIQ/SUBSPIQ); no longer U1.18 (GPIO10/TOUCH10/ADC1_CH9/FSPICS0/FSPIIO4/SUBSPICS0)
- net ISO_PWM_M2: now also U1.29 (SPIIO7/GPIO36/FSPICLK/SUBSPICLK); no longer U1.19 (GPIO11/TOUCH11/ADC2_CH0/FSPID/FSPIIO5/SUBSPID)
- net ISO_PWM_M3: now also U1.28 (SPIIO6/GPIO35/FSPID/SUBSPID); no longer U1.20 (GPIO12/TOUCH12/ADC2_CH1/FSPICLK/FSPIIO6/SUBSPICLK)
- net ISO_PWM_M4: now also U1.26 (GPIO45); no longer U1.21 (GPIO13/TOUCH13/ADC2_CH2/FSPIQ/FSPIIO7/SUBSPIQ)
- net ISO_STBY: now also U1.31 (GPIO38/FSPIWP/SUBSPIWP); no longer U1.17 (GPIO9/TOUCH9/ADC1_CH8/FSPIHD/SUBSPIHD)
Changed lines of the file:
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@@
 	)
 	(no_connect
-		(at 160.02 59.69)
+		(at 160.02 92.71)
+	)
+	(no_connect
+		(at 160.02 82.55)
 	)
 	(no_connect
@@
 	)
 	(no_connect
-		(at 160.02 118.11)
-	)
-	(no_connect
-		(at 68.58 74.93)
+		(at 160.02 87.63)
 	)
 	(no_connect
@@
 	)
 	(no_connect
+		(at 160.02 105.41)
+	)
+	(no_connect
 		(at 160.02 128.27)
 	)
 	(no_connect
+		(at 160.02 80.01)
+	)
+	(no_connect
+		(at 160.02 85.09)
+	)
+	(no_connect
+		(at 160.02 100.33)
+	)
+	(no_connect
 		(at 160.02 123.19)
 	)
 	(no_connect
-		(at 68.58 80.01)
-	)
-	(no_connect
-		(at 160.02 120.65)
-	)
-	(no_connect
-		(at 68.58 72.39)
-	)
-	(no_connect
-		(at 68.58 77.47)
-	)
-	(no_connect
-		(at 68.58 125.73)
-	)
-	(no_connect
-		(at 160.02 57.15)
+		(at 160.02 102.87)
+	)
+	(no_connect
+		(at 160.02 95.25)
+	)
+	(no_connect
+		(at 160.02 97.79)
 	)
 	(no_connect
@@
 	)
 	(no_connect
+		(at 160.02 90.17)
+	)
+	(no_connect
 		(at 160.02 115.57)
 	)
-	(no_connect
-		(at 68.58 128.27)
-	)
-	(no_connect
-		(at 68.58 123.19)
-	)
 	(wire
 		(pts
@@
 		)
 	)
+	(hierarchical_label "GPIO15"
+		(shape input)
+		(at 68.58 64.77 180)
+		(effects
+			(font
+				(size 1.27 1.27)
+			)
+			(justify right)
+		)
+	)
+	(hierarchical_label "ISO_M2_CLOSE"
+		(shape input)
+		(at 160.02 59.69 0)
+		(effects
+			(font
+				(size 1.27 1.27)
+			)
+			(justify left)
+		)
+	)
+	(hierarchical_label "GPIO19"
+		(shape input)
+		(at 160.02 67.31 0)
+		(effects
+			(font
+				(size 1.27 1.27)
+			)
+			(justify left)
+		)
+	)
+	(hierarchical_label "ISO_M4_OPEN"
+		(shape input)
+		(at 68.58 74.93 180)
+		(effects
+			(font
+				(size 1.27 1.27)
+			)
+			(justify right)
+		)
+	)
+	(hierarchical_label "ISO_PWM_M3"
+		(shape input)
+		(at 68.58 123.19 180)
+		(effects
+			(font
+				(size 1.27 1.27)
+			)
+			(justify right)
+		)
+	)
+	(hierarchical_label "ISO_STBY"
+		(shape input)
+		(at 160.02 118.11 0)
+		(effects
+			(font
+				(size 1.27 1.27)
+			)
+			(justify left)
+		)
+	)
+	(hierarchical_label "ISO_M1_CLOSE"
+		(shape input)
+		(at 160.02 77.47 0)
+		(effects
+			(font
+				(size 1.27 1.27)
+			)
+			(justify left)
+		)
+	)
+	(hierarchical_label "ISO_M2_OPEN"
+		(shape input)
+		(at 160.02 57.15 0)
+		(effects
+			(font
+				(size 1.27 1.27)
+			)
+			(justify left)
+		)
+	)
+	(hierarchical_label "ISO_M1_OPEN"
+		(shape input)
+		(at 160.02 74.93 0)
+		(effects
+			(font
+				(size 1.27 1.27)
+			)
+			(justify left)
+		)
+	)
 	(hierarchical_label "ISO_PWM_M4"
 		(shape input)
-		(at 160.02 105.41 0)
-		(effects
-			(font
-				(size 1.27 1.27)
-			)
-			(justify left)
+		(at 160.02 120.65 0)
+		(effects
+			(font
+				(size 1.27 1.27)
+			)
+			(justify left)
+		)
+	)
+	(hierarchical_label "ISO_PWM_M1"
+		(shape input)
+		(at 68.58 128.27 180)
+		(effects
+			(font
+				(size 1.27 1.27)
+			)
+			(justify right)
 		)
 	)
 	(hierarchical_label "ISO_M3_CLOSE"
 		(shape input)
-		(at 160.02 87.63 0)
-		(effects
-			(font
-				(size 1.27 1.27)
-			)
-			(justify left)
-		)
-	)
-	(hierarchical_label "GPIO15"
-		(shape input)
-		(at 68.58 64.77 180)
-		(effects
-			(font
-				(size 1.27 1.27)
-			)
-			(justify right)
-		)
-	)
-	(hierarchical_label "GPIO19"
-		(shape input)
-		(at 160.02 67.31 0)
-		(effects
-			(font
-				(size 1.27 1.27)
-			)
-			(justify left)
+		(at 68.58 77.47 180)
+		(effects
+			(font
+				(size 1.27 1.27)
+			)
+			(justify right)
 		)
 	)
 	(hierarchical_label "ISO_M4_CLOSE"
 		(shape input)
-		(at 160.02 92.71 0)
-		(effects
-			(font
-				(size 1.27 1.27)
-			)
-			(justify left)
-		)
-	)
-	(hierarchical_label "ISO_STBY"
-		(shape input)
-		(at 160.02 95.25 0)
-		(effects
-			(font
-				(size 1.27 1.27)
-			)
-			(justify left)
-		)
-	)
-	(hierarchical_label "ISO_M1_CLOSE"
-		(shape input)
-		(at 160.02 77.47 0)
-		(effects
-			(font
-				(size 1.27 1.27)
-			)
-			(justify left)
-		)
-	)
-	(hierarchical_label "ISO_M4_OPEN"
-		(shape input)
-		(at 160.02 90.17 0)
-		(effects
-			(font
-				(size 1.27 1.27)
-			)
-			(justify left)
-		)
-	)
-	(hierarchical_label "ISO_PWM_M3"
-		(shape input)
-		(at 160.02 102.87 0)
+		(at 68.58 72.39 180)
+		(effects
+			(font
+				(size 1.27 1.27)
+			)
+			(justify right)
+		)
+	)
+	(hierarchical_label "GPIO20"
+		(shape input)
+		(at 160.02 64.77 0)
 		(effects
 			(font
@@
 	(hierarchical_label "ISO_PWM_M2"
 		(shape input)
-		(at 160.02 100.33 0)
-		(effects
-			(font
-				(size 1.27 1.27)
-			)
-			(justify left)
-		)
-	)
-	(hierarchical_label "ISO_M1_OPEN"
-		(shape input)
-		(at 160.02 74.93 0)
-		(effects
-			(font
-				(size 1.27 1.27)
-			)
-			(justify left)
-		)
-	)
-	(hierarchical_label "GPIO20"
-		(shape input)
-		(at 160.02 64.77 0)
-		(effects
-			(font
-				(size 1.27 1.27)
-			)
-			(justify left)
-		)
-	)
-	(hierarchical_label "ISO_M2_CLOSE"
-		(shape input)
-		(at 160.02 82.55 0)
-		(effects
-			(font
-				(size 1.27 1.27)
-			)
-			(justify left)
-		)
-	)
-	(hierarchical_label "ISO_M2_OPEN"
-		(shape input)
-		(at 160.02 80.01 0)
-		(effects
-			(font
-				(size 1.27 1.27)
-			)
-			(justify left)
-		)
-	)
-	(hierarchical_label "ISO_PWM_M1"
-		(shape input)
-		(at 160.02 97.79 0)
-		(effects
-			(font
-				(size 1.27 1.27)
-			)
-			(justify left)
+		(at 68.58 125.73 180)
+		(effects
+			(font
+				(size 1.27 1.27)
+			)
+			(justify right)
 		)
 	)
 	(hierarchical_label "ISO_M3_OPEN"
 		(shape input)
-		(at 160.02 85.09 0)
-		(effects
-			(font
-				(size 1.27 1.27)
-			)
-			(justify left)
-		)
-	)
+		(at 68.58 80.01 180)
+		(effects
+			(font
+				(size 1.27 1.27)
+			)
+			(justify right)
+		)
+	)

Commit message: PCB tracing complete
Connections:
- net ISO_M2_CLOSE: now also U1.35 (MTMS/GPIO42); no longer U1.36 (U0RXD/GPIO44/CLK_OUT2)
- net ISO_M2_OPEN: now also U1.36 (U0RXD/GPIO44/CLK_OUT2); no longer U1.37 (U0TXD/GPIO43/CLK_OUT1)
- net ISO_M3_CLOSE: now also U1.32 (MTCK/GPIO39/CLK_OUT3/SUBSPICS1); no longer U1.34 (MTDI/GPIO41/CLK_OUT1)
- net ISO_M3_OPEN: now also U1.31 (GPIO38/FSPIWP/SUBSPIWP); no longer U1.35 (MTMS/GPIO42)
- net ISO_M4_CLOSE: now also U1.29 (SPIIO7/GPIO36/FSPICLK/SUBSPICLK); no longer U1.32 (MTCK/GPIO39/CLK_OUT3/SUBSPICS1)
- net ISO_M4_OPEN: now also U1.30 (SPIDQS/GPIO37/FSPIQ/SUBSPIQ); no longer U1.33 (MTDO/GPIO40/CLK_OUT2)
- net ISO_PWM_M1: now also U1.37 (U0TXD/GPIO43/CLK_OUT1); no longer U1.30 (SPIDQS/GPIO37/FSPIQ/SUBSPIQ)
- net ISO_PWM_M2: now also U1.34 (MTDI/GPIO41/CLK_OUT1); no longer U1.29 (SPIIO7/GPIO36/FSPICLK/SUBSPICLK)
- net ISO_PWM_M3: now also U1.33 (MTDO/GPIO40/CLK_OUT2); no longer U1.28 (SPIIO6/GPIO35/FSPID/SUBSPID)
- net ISO_PWM_M4: now also U1.28 (SPIIO6/GPIO35/FSPID/SUBSPID); no longer U1.26 (GPIO45)
- net ISO_STBY: now also U1.26 (GPIO45); no longer U1.31 (GPIO38/FSPIWP/SUBSPIWP)
Changed lines of the file:
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@@
-		)
-	)
-	(hierarchical_label "ISO_M2_CLOSE"
-		(shape input)
-		(at 160.02 59.69 0)
-		(effects
-			(font
-				(size 1.27 1.27)
-			)
-			(justify left)
 		)
 	)
@@
 		)
 	)
-	(hierarchical_label "ISO_M4_OPEN"
-		(shape input)
-		(at 68.58 74.93 180)
-		(effects
-			(font
-				(size 1.27 1.27)
-			)
-			(justify right)
-		)
-	)
-	(hierarchical_label "ISO_PWM_M3"
+	(hierarchical_label "ISO_PWM_M4"
 		(shape input)
 		(at 68.58 123.19 180)
@@
 			)
 			(justify right)
-		)
-	)
-	(hierarchical_label "ISO_STBY"
-		(shape input)
-		(at 160.02 118.11 0)
-		(effects
-			(font
-				(size 1.27 1.27)
-			)
-			(justify left)
 		)
 	)
@@
 		)
 	)
+	(hierarchical_label "ISO_PWM_M1"
+		(shape input)
+		(at 160.02 57.15 0)
+		(effects
+			(font
+				(size 1.27 1.27)
+			)
+			(justify left)
+		)
+	)
+	(hierarchical_label "ISO_M4_OPEN"
+		(shape input)
+		(at 68.58 128.27 180)
+		(effects
+			(font
+				(size 1.27 1.27)
+			)
+			(justify right)
+		)
+	)
 	(hierarchical_label "ISO_M2_OPEN"
 		(shape input)
-		(at 160.02 57.15 0)
+		(at 160.02 59.69 0)
 		(effects
 			(font
@@
 		)
 	)
-	(hierarchical_label "ISO_PWM_M4"
+	(hierarchical_label "ISO_M2_CLOSE"
 		(shape input)
-		(at 160.02 120.65 0)
-		(effects
-			(font
-				(size 1.27 1.27)
-			)
-			(justify left)
-		)
-	)
-	(hierarchical_label "ISO_PWM_M1"
-		(shape input)
-		(at 68.58 128.27 180)
+		(at 68.58 80.01 180)
 		(effects
 			(font
@@
 		)
 	)
-	(hierarchical_label "ISO_M3_CLOSE"
+	(hierarchical_label "ISO_PWM_M2"
 		(shape input)
 		(at 68.58 77.47 180)
@@
 		)
 	)
-	(hierarchical_label "ISO_M4_CLOSE"
+	(hierarchical_label "ISO_M3_OPEN"
+		(shape input)
+		(at 160.02 118.11 0)
+		(effects
+			(font
+				(size 1.27 1.27)
+			)
+			(justify left)
+		)
+	)
+	(hierarchical_label "ISO_M3_CLOSE"
 		(shape input)
 		(at 68.58 72.39 180)
+		(effects
+			(font
+				(size 1.27 1.27)
+			)
+			(justify right)
+		)
+	)
+	(hierarchical_label "ISO_PWM_M3"
+		(shape input)
+		(at 68.58 74.93 180)
 		(effects
 			(font
@@
 		)
 	)
-	(hierarchical_label "ISO_PWM_M2"
+	(hierarchical_label "ISO_M4_CLOSE"
 		(shape input)
 		(at 68.58 125.73 180)
@@
 		)
 	)
-	(hierarchical_label "ISO_M3_OPEN"
+	(hierarchical_label "ISO_STBY"
 		(shape input)
-		(at 68.58 80.01 180)
+		(at 160.02 120.65 0)
 		(effects
 			(font
 				(size 1.27 1.27)
 			)
-			(justify right)
+			(justify left)
 		)
 	)

Commit message: BOM work
Parts:
- C7: renamed from C34; LCSC (none) -> C1590
- C8: renamed from C33; value 10uF -> 10uF 10V; LCSC (none) -> C17024
- R5: renamed from R2; LCSC (none) -> C25804
- R_BOOT1: LCSC (none) -> C25804
- R_LED1: value 470R -> 330R; LCSC (none) -> C23138
- SW1: renamed from SW2; LCSC (none) -> C51927445
- SW2: renamed from SW1; LCSC (none) -> C51927445
- U3: renamed from U1; LCSC (none) -> C2913197
Changed lines of the file:
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@@
 		(dnp no)
 		(fields_autoplaced yes)
-		(property "Reference" "C34"
+		(property "Reference" "C7"
 			(at 118.11 26.67 90)
 			(effects
@@
 			)
 		)
+		(property "LCSC" "C1590"
+			(at 118.11 34.29 90)
+			(effects
+				(font
+					(size 1.27 1.27)
+				)
+				(hide yes)
+			)
+		)
 		(pin "2"
 		)
@@
 			(project "barn-blinds-controller"
 				(path "/aa90962a-81b9-423d-8acd-c4e83fa798bb/3a264230-9604-4127-a232-ac76a818f339"
-					(reference "C34")
+					(reference "C7")
 					(unit 1)
 				)
@@
 		(dnp no)
 		(fields_autoplaced yes)
-		(property "Reference" "SW2"
+		(property "Reference" "SW1"
 			(at 60.96 48.26 0)
 			(effects
@@
 			)
 		)
+		(property "LCSC" "C51927445"
+			(at 60.96 54.61 0)
+			(effects
+				(font
+					(size 1.27 1.27)
+				)
+				(hide yes)
+			)
+		)
 		(pin "1"
 		)
@@
 			(project "barn-blinds-controller"
 				(path "/aa90962a-81b9-423d-8acd-c4e83fa798bb/3a264230-9604-4127-a232-ac76a818f339"
-					(reference "SW2")
+					(reference "SW1")
 					(unit 1)
 				)
@@
 			)
 		)
-		(property "Value" "470R"
+		(property "Value" "330R"
 			(at 48.26 64.77 90)
 			(effects
@@
 			)
 		)
+		(property "LCSC" "C23138"
+			(at 48.26 68.58 90)
+			(effects
+				(font
+					(size 1.27 1.27)
+				)
+				(hide yes)
+			)
+		)
 		(pin "2"
 		)
@@
 		(dnp no)
 		(fields_autoplaced yes)
-		(property "Reference" "U1"
+		(property "Reference" "U3"
 			(at 116.4433 49.53 0)
 			(effects
@@
 			)
 		)
+		(property "LCSC" "C2913197"
+			(at 114.3 92.71 0)
+			(effects
+				(font
+					(size 1.27 1.27)
+				)
+				(hide yes)
+			)
+		)
 		(pin "19"
 		)
@@
 			(project "barn-blinds-controller"
 				(path "/aa90962a-81b9-423d-8acd-c4e83fa798bb/3a264230-9604-4127-a232-ac76a818f339"
-					(reference "U1")
+					(reference "U3")
 					(unit 1)
 				)
@@
 		(dnp no)
 		(fields_autoplaced yes)
-		(property "Reference" "C33"
+		(property "Reference" "C8"
 			(at 117.221 38.1 90)
 			(effects
@@
 			)
 		)
-		(property "Value" "10uF"
+		(property "Value" "10uF 10V"
 			(at 117.221 40.64 90)
 			(effects
@@
 			)
 		)
+		(property "LCSC" "C17024"
+			(at 118.11 45.72 90)
+			(effects
+				(font
+					(size 1.27 1.27)
+				)
+				(hide yes)
+			)
+		)
 		(pin "2"
 		)
@@
 			(project "barn-blinds-controller"
 				(path "/aa90962a-81b9-423d-8acd-c4e83fa798bb/3a264230-9604-4127-a232-ac76a818f339"
-					(reference "C33")
+					(reference "C8")
 					(unit 1)
 				)
@@
 		(dnp no)
 		(fields_autoplaced yes)
-		(property "Reference" "#PWR053"
+		(property "Reference" "#PWR022"
 			(at 128.27 45.72 0)
 			(effects
@@
 			(project "barn-blinds-controller"
 				(path "/aa90962a-81b9-423d-8acd-c4e83fa798bb/3a264230-9604-4127-a232-ac76a818f339"
-					(reference "#PWR053")
+					(reference "#PWR022")
 					(unit 1)
 				)
@@
 		(dnp no)
 		(fields_autoplaced yes)
-		(property "Reference" "#PWR041"
+		(property "Reference" "#PWR019"
 			(at 114.3 34.29 0)
 			(effects
@@
 			(project "barn-blinds-controller"
 				(path "/aa90962a-81b9-423d-8acd-c4e83fa798bb/3a264230-9604-4127-a232-ac76a818f339"
-					(reference "#PWR041")
+					(reference "#PWR019")
 					(unit 1)
 				)
@@
 			)
 		)
+		(property "LCSC" "C25804"
+			(at 182.88 76.2 0)
+			(effects
+				(font
+					(size 1.27 1.27)
+				)
+				(hide yes)
+			)
+		)
 		(pin "2"
 		)
@@
 		(dnp no)
 		(fields_autoplaced yes)
-		(property "Reference" "SW1"
+		(property "Reference" "SW2"
 			(at 203.2 66.04 0)
 			(effects
@@
 			)
 		)
+		(property "LCSC" "C51927445"
+			(at 203.2 72.39 0)
+			(effects
+				(font
+					(size 1.27 1.27)
+				)
+				(hide yes)
+			)
+		)
 		(pin "1"
 		)
@@
 			(project "barn-blinds-controller"
 				(path "/aa90962a-81b9-423d-8acd-c4e83fa798bb/3a264230-9604-4127-a232-ac76a818f339"
-					(reference "SW1")
+					(reference "SW2")
 					(unit 1)
 				)
@@
 		(dnp no)
 		(fields_autoplaced yes)
-		(property "Reference" "#PWR047"
+		(property "Reference" "#PWR020"
 			(at 114.3 139.7 0)
 			(effects
@@
 			(project "barn-blinds-controller"
 				(path "/aa90962a-81b9-423d-8acd-c4e83fa798bb/3a264230-9604-4127-a232-ac76a818f339"
-					(reference "#PWR047")
+					(reference "#PWR020")
 					(unit 1)
 				)
@@
 		(dnp no)
 		(fields_autoplaced yes)
-		(property "Reference" "#PWR054"
+		(property "Reference" "#PWR021"
 			(at 128.27 34.29 0)
 			(effects
@@
 			(project "barn-blinds-controller"
 				(path "/aa90962a-81b9-423d-8acd-c4e83fa798bb/3a264230-9604-4127-a232-ac76a818f339"
-					(reference "#PWR054")
+					(reference "#PWR021")
 					(unit 1)
 				)
@@
 		(dnp no)
 		(fields_autoplaced yes)
-		(property "Reference" "#PWR048"
+		(property "Reference" "#PWR018"
 			(at 66.04 46.99 0)
 			(effects
@@
 			(project "barn-blinds-controller"
 				(path "/aa90962a-81b9-423d-8acd-c4e83fa798bb/3a264230-9604-4127-a232-ac76a818f339"
-					(reference "#PWR048")
+					(reference "#PWR018")
 					(unit 1)
 				)
@@
 		(dnp no)
 		(fields_autoplaced yes)
-		(property "Reference" "R2"
+		(property "Reference" "R5"
 			(at 68.58 45.7199 0)
 			(effects
@@
 			)
 		)
+		(property "LCSC" "C25804"
+			(at 66.04 46.99 0)
+			(effects
+				(font
+					(size 1.27 1.27)
+				)
+				(hide yes)
+			)
+		)
 		(pin "2"
 		)
@@
 			(project "barn-blinds-controller"
 				(path "/aa90962a-81b9-423d-8acd-c4e83fa798bb/3a264230-9604-4127-a232-ac76a818f339"
-					(reference "R2")
+					(reference "R5")
 					(unit 1)
 				)
@@
 		(dnp no)
 		(fields_autoplaced yes)
-		(property "Reference" "#PWR052"
+		(property "Reference" "#PWR016"
 			(at 44.45 82.55 0)
 			(effects
@@
 			(project "barn-blinds-controller"
 				(path "/aa90962a-81b9-423d-8acd-c4e83fa798bb/3a264230-9604-4127-a232-ac76a818f339"
-					(reference "#PWR052")
+					(reference "#PWR016")
 					(unit 1)
 				)
@@
 		(dnp no)
 		(fields_autoplaced yes)
-		(property "Reference" "#PWR049"
+		(property "Reference" "#PWR017"
 			(at 45.72 57.15 0)
 			(effects
@@
 			(project "barn-blinds-controller"
 				(path "/aa90962a-81b9-423d-8acd-c4e83fa798bb/3a264230-9604-4127-a232-ac76a818f339"
-					(reference "#PWR049")
+					(reference "#PWR017")
 					(unit 1)
 				)
@@
 		(dnp no)
 		(fields_autoplaced yes)
-		(property "Reference" "#PWR051"
+		(property "Reference" "#PWR023"
 			(at 182.88 76.2 0)
 			(effects
@@
 			(project "barn-blinds-controller"
 				(path "/aa90962a-81b9-423d-8acd-c4e83fa798bb/3a264230-9604-4127-a232-ac76a818f339"
-					(reference "#PWR051")
+					(reference "#PWR023")
 					(unit 1)
 				)
@@
 		(dnp no)
 		(fields_autoplaced yes)
-		(property "Reference" "#PWR050"
+		(property "Reference" "#PWR024"
 			(at 228.6 74.93 0)
 			(effects
@@
 			(project "barn-blinds-controller"
 				(path "/aa90962a-81b9-423d-8acd-c4e83fa798bb/3a264230-9604-4127-a232-ac76a818f339"
-					(reference "#PWR050")
-					(unit 1)
-				)
+					(reference "#PWR024")
+					(unit 1)
+				)

Commit message: Refactored board to use larger vias and route better paths.
Connections:
- net ISO_M1_CLOSE: now also U3.35 (MTMS/GPIO42); no longer U3.38 (GPIO2/TOUCH2/ADC1_CH1)
- net ISO_M1_OPEN: now also U3.36 (U0RXD/GPIO44/CLK_OUT2); no longer U3.39 (GPIO1/TOUCH1/ADC1_CH0)
- net ISO_M2_CLOSE: now also U3.38 (GPIO2/TOUCH2/ADC1_CH1); no longer U3.35 (MTMS/GPIO42)
- net ISO_M2_OPEN: now also U3.37 (U0TXD/GPIO43/CLK_OUT1); no longer U3.36 (U0RXD/GPIO44/CLK_OUT2)
- net ISO_M3_CLOSE: now also U3.28 (SPIIO6/GPIO35/FSPID/SUBSPID); no longer U3.32 (MTCK/GPIO39/CLK_OUT3/SUBSPICS1)
- net ISO_M3_OPEN: now also U3.29 (SPIIO7/GPIO36/FSPICLK/SUBSPICLK); no longer U3.31 (GPIO38/FSPIWP/SUBSPIWP)
- net ISO_M4_CLOSE: now also U3.32 (MTCK/GPIO39/CLK_OUT3/SUBSPICS1); no longer U3.29 (SPIIO7/GPIO36/FSPICLK/SUBSPICLK)
- net ISO_M4_OPEN: now also U3.31 (GPIO38/FSPIWP/SUBSPIWP); no longer U3.30 (SPIDQS/GPIO37/FSPIQ/SUBSPIQ)
- net ISO_PWM_M1: now also U3.34 (MTDI/GPIO41/CLK_OUT1); no longer U3.37 (U0TXD/GPIO43/CLK_OUT1)
- net ISO_PWM_M2: now also U3.39 (GPIO1/TOUCH1/ADC1_CH0); no longer U3.34 (MTDI/GPIO41/CLK_OUT1)
- net ISO_PWM_M3: now also U3.26 (GPIO45); no longer U3.33 (MTDO/GPIO40/CLK_OUT2)
- net ISO_PWM_M4: now also U3.33 (MTDO/GPIO40/CLK_OUT2); no longer U3.28 (SPIIO6/GPIO35/FSPID/SUBSPID)
- net ISO_STBY: now also U3.30 (SPIDQS/GPIO37/FSPIQ/SUBSPIQ); no longer U3.26 (GPIO45)
Changed lines of the file:
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@@
+		)
+	)
+	(hierarchical_label "ISO_M1_CLOSE"
+		(shape input)
+		(at 68.58 80.01 180)
+		(effects
+			(font
+				(size 1.27 1.27)
+			)
+			(justify right)
+		)
+	)
+	(hierarchical_label "ISO_M2_OPEN"
+		(shape input)
+		(at 160.02 57.15 0)
+		(effects
+			(font
+				(size 1.27 1.27)
+			)
+			(justify left)
+		)
+	)
+	(hierarchical_label "ISO_PWM_M1"
+		(shape input)
+		(at 68.58 77.47 180)
+		(effects
+			(font
+				(size 1.27 1.27)
+			)
+			(justify right)
 		)
 	)
@@
 		)
 	)
-	(hierarchical_label "ISO_PWM_M4"
+	(hierarchical_label "ISO_M3_CLOSE"
 		(shape input)
 		(at 68.58 123.19 180)
@@
 		)
 	)
-	(hierarchical_label "ISO_M1_CLOSE"
+	(hierarchical_label "ISO_PWM_M3"
+		(shape input)
+		(at 160.02 120.65 0)
+		(effects
+			(font
+				(size 1.27 1.27)
+			)
+			(justify left)
+		)
+	)
+	(hierarchical_label "ISO_PWM_M4"
+		(shape input)
+		(at 68.58 74.93 180)
+		(effects
+			(font
+				(size 1.27 1.27)
+			)
+			(justify right)
+		)
+	)
+	(hierarchical_label "ISO_M4_CLOSE"
+		(shape input)
+		(at 68.58 72.39 180)
+		(effects
+			(font
+				(size 1.27 1.27)
+			)
+			(justify right)
+		)
+	)
+	(hierarchical_label "ISO_M2_CLOSE"
 		(shape input)
 		(at 160.02 77.47 0)
@@
 		)
 	)
-	(hierarchical_label "ISO_PWM_M1"
-		(shape input)
-		(at 160.02 57.15 0)
-		(effects
-			(font
-				(size 1.27 1.27)
-			)
-			(justify left)
-		)
-	)
-	(hierarchical_label "ISO_M4_OPEN"
+	(hierarchical_label "ISO_STBY"
 		(shape input)
 		(at 68.58 128.27 180)
@@
 		)
 	)
-	(hierarchical_label "ISO_M2_OPEN"
+	(hierarchical_label "ISO_M4_OPEN"
 		(shape input)
-		(at 160.02 59.69 0)
+		(at 160.02 118.11 0)
+		(effects
+			(font
+				(size 1.27 1.27)
+			)
+			(justify left)
+		)
+	)
+	(hierarchical_label "ISO_PWM_M2"
+		(shape input)
+		(at 160.02 74.93 0)
 		(effects
 			(font
@@
 	(hierarchical_label "ISO_M1_OPEN"
 		(shape input)
-		(at 160.02 74.93 0)
+		(at 160.02 59.69 0)
 		(effects
 			(font
@@
 			)
 			(justify left)
-		)
-	)
-	(hierarchical_label "ISO_M2_CLOSE"
-		(shape input)
-		(at 68.58 80.01 180)
-		(effects
-			(font
-				(size 1.27 1.27)
-			)
-			(justify right)
-		)
-	)
-	(hierarchical_label "ISO_PWM_M2"
-		(shape input)
-		(at 68.58 77.47 180)
-		(effects
-			(font
-				(size 1.27 1.27)
-			)
-			(justify right)
-		)
-	)
-	(hierarchical_label "ISO_M3_OPEN"
-		(shape input)
-		(at 160.02 118.11 0)
-		(effects
-			(font
-				(size 1.27 1.27)
-			)
-			(justify left)
-		)
-	)
-	(hierarchical_label "ISO_M3_CLOSE"
-		(shape input)
-		(at 68.58 72.39 180)
-		(effects
-			(font
-				(size 1.27 1.27)
-			)
-			(justify right)
-		)
-	)
-	(hierarchical_label "ISO_PWM_M3"
-		(shape input)
-		(at 68.58 74.93 180)
-		(effects
-			(font
-				(size 1.27 1.27)
-			)
-			(justify right)
 		)
 	)
@@
 		)
 	)
-	(hierarchical_label "ISO_M4_CLOSE"
+	(hierarchical_label "ISO_M3_OPEN"
 		(shape input)
 		(at 68.58 125.73 180)
@@
 		)
 	)
-	(hierarchical_label "ISO_STBY"
-		(shape input)
-		(at 160.02 120.65 0)
-		(effects
-			(font
-				(size 1.27 1.27)
-			)
-			(justify left)
-		)
-	)
