File: sensors.kicad_sch (KiCad schematic)
At the start: 6 parts, among them U10 ACS723xLCTR-05AB, U11 TMP235

Commit message: BOM work
Parts:
- C_ACS1, C_TMP1: LCSC (none) -> C1590
- C_ACS2: value 10nF -> 10nF 10V; LCSC (none) -> C519405
- C_FILT1: value 1nF -> 1nF 10V; LCSC (none) -> C519402
- U10: renamed from U11; LCSC (none) -> C2861437
- U11: renamed from U10; LCSC (none) -> C2655492
Connections:
- no-connect marks 0 -> 2
Changed lines of the file:
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@@
 		(color 0 0 0 0)
+	)
+	(no_connect
+		(at 91.44 87.63)
+	)
+	(no_connect
+		(at 71.12 85.09)
 	)
 	(wire
@@
 			)
 		)
-		(property "Value" "10nF"
+		(property "Value" "10nF 10V"
 			(at 114.3 48.2599 0)
 			(effects
@@
 			)
 		)
+		(property "LCSC" "C519405"
+			(at 110.49 46.99 0)
+			(effects
+				(font
+					(size 1.27 1.27)
+				)
+				(hide yes)
+			)
+		)
 		(pin "1"
 		)
@@
 		(dnp no)
 		(fields_autoplaced yes)
-		(property "Reference" "#PWR082"
+		(property "Reference" "#PWR083"
 			(at 97.79 29.21 0)
 			(effects
@@
 			(project "barn-blinds-controller"
 				(path "/aa90962a-81b9-423d-8acd-c4e83fa798bb/8f0cb6d8-027e-4edb-b8ea-04d7ddb83db1"
-					(reference "#PWR082")
+					(reference "#PWR083")
 					(unit 1)
 				)
@@
 			)
 		)
+		(property "LCSC" "C1590"
+			(at 87.63 29.21 90)
+			(effects
+				(font
+					(size 1.27 1.27)
+				)
+				(hide yes)
+			)
+		)
 		(pin "1"
 		)
@@
 		(dnp no)
 		(fields_autoplaced yes)
-		(property "Reference" "#PWR087"
+		(property "Reference" "#PWR085"
 			(at 99.06 99.06 0)
 			(effects
@@
 			(project "barn-blinds-controller"
 				(path "/aa90962a-81b9-423d-8acd-c4e83fa798bb/8f0cb6d8-027e-4edb-b8ea-04d7ddb83db1"
-					(reference "#PWR087")
+					(reference "#PWR085")
 					(unit 1)
 				)
@@
 		(dnp no)
 		(fields_autoplaced yes)
-		(property "Reference" "#PWR081"
+		(property "Reference" "#PWR084"
 			(at 97.79 64.77 0)
 			(effects
@@
 			(project "barn-blinds-controller"
 				(path "/aa90962a-81b9-423d-8acd-c4e83fa798bb/8f0cb6d8-027e-4edb-b8ea-04d7ddb83db1"
-					(reference "#PWR081")
+					(reference "#PWR084")
 					(unit 1)
 				)
@@
 		(dnp no)
 		(fields_autoplaced yes)
-		(property "Reference" "#PWR078"
+		(property "Reference" "#PWR079"
 			(at 77.47 43.18 0)
 			(effects
@@
 			(project "barn-blinds-controller"
 				(path "/aa90962a-81b9-423d-8acd-c4e83fa798bb/8f0cb6d8-027e-4edb-b8ea-04d7ddb83db1"
-					(reference "#PWR078")
+					(reference "#PWR079")
 					(unit 1)
 				)
@@
 		(dnp no)
 		(fields_autoplaced yes)
-		(property "Reference" "#PWR083"
+		(property "Reference" "#PWR087"
 			(at 110.49 57.15 0)
 			(effects
@@
 			(project "barn-blinds-controller"
 				(path "/aa90962a-81b9-423d-8acd-c4e83fa798bb/8f0cb6d8-027e-4edb-b8ea-04d7ddb83db1"
-					(reference "#PWR083")
+					(reference "#PWR087")
 					(unit 1)
 				)
@@
 		(dnp no)
 		(fields_autoplaced yes)
-		(property "Reference" "#PWR086"
+		(property "Reference" "#PWR078"
 			(at 64.77 87.63 0)
 			(effects
@@
 			(project "barn-blinds-controller"
 				(path "/aa90962a-81b9-423d-8acd-c4e83fa798bb/8f0cb6d8-027e-4edb-b8ea-04d7ddb83db1"
-					(reference "#PWR086")
+					(reference "#PWR078")
 					(unit 1)
 				)
@@
 		(dnp no)
 		(fields_autoplaced yes)
-		(property "Reference" "#PWR085"
+		(property "Reference" "#PWR086"
 			(at 100.33 85.09 0)
 			(effects
@@
 			(project "barn-blinds-controller"
 				(path "/aa90962a-81b9-423d-8acd-c4e83fa798bb/8f0cb6d8-027e-4edb-b8ea-04d7ddb83db1"
-					(reference "#PWR085")
+					(reference "#PWR086")
 					(unit 1)
 				)
@@
 		(dnp no)
 		(fields_autoplaced yes)
-		(property "Reference" "#PWR084"
+		(property "Reference" "#PWR080"
 			(at 77.47 50.8 0)
 			(effects
@@
 			(project "barn-blinds-controller"
 				(path "/aa90962a-81b9-423d-8acd-c4e83fa798bb/8f0cb6d8-027e-4edb-b8ea-04d7ddb83db1"
-					(reference "#PWR084")
+					(reference "#PWR080")
 					(unit 1)
 				)
@@
 		(dnp no)
 		(fields_autoplaced yes)
-		(property "Reference" "U11"
+		(property "Reference" "U10"
 			(at 81.28 77.47 0)
 			(effects
@@
 			)
 		)
+		(property "LCSC" "C2861437"
+			(at 73.66 86.36 0)
+			(effects
+				(font
+					(size 1.27 1.27)
+				)
+				(hide yes)
+			)
+		)
 		(pin "5"
 		)
@@
 			(project "barn-blinds-controller"
 				(path "/aa90962a-81b9-423d-8acd-c4e83fa798bb/8f0cb6d8-027e-4edb-b8ea-04d7ddb83db1"
-					(reference "U11")
+					(reference "U10")
 					(unit 1)
 				)
@@
 		(dnp no)
 		(fields_autoplaced yes)
-		(property "Reference" "#PWR080"
+		(property "Reference" "#PWR082"
 			(at 83.82 64.77 0)
 			(effects
@@
 			(project "barn-blinds-controller"
 				(path "/aa90962a-81b9-423d-8acd-c4e83fa798bb/8f0cb6d8-027e-4edb-b8ea-04d7ddb83db1"
-					(reference "#PWR080")
+					(reference "#PWR082")
 					(unit 1)
 				)
@@
 			)
 		)
-		(property "Value" "1nF"
+		(property "Value" "1nF 10V"
 			(at 101.6 55.8799 0)
 			(effects
@@
 			)
 		)
+		(property "LCSC" "C519402"
+			(at 97.79 54.61 0)
+			(effects
+				(font
+					(size 1.27 1.27)
+				)
+				(hide yes)
+			)
+		)
 		(pin "2"
 		)
@@
 			)
 		)
+		(property "LCSC" "C1590"
+			(at 99.06 88.9 0)
+			(effects
+				(font
+					(size 1.27 1.27)
+				)
+				(hide yes)
+			)
+		)
 		(pin "2"
 		)
@@
 		(dnp no)
 		(fields_autoplaced yes)
-		(property "Reference" "U10"
+		(property "Reference" "U11"
 			(at 85.9633 35.56 0)
 			(effects
@@
 			)
 		)
+		(property "LCSC" "C2655492"
+			(at 83.82 48.26 0)
+			(effects
+				(font
+					(size 1.27 1.27)
+				)
+				(hide yes)
+			)
+		)
 		(pin "6"
 		)
@@
 			(project "barn-blinds-controller"
 				(path "/aa90962a-81b9-423d-8acd-c4e83fa798bb/8f0cb6d8-027e-4edb-b8ea-04d7ddb83db1"
-					(reference "U10")
+					(reference "U11")
 					(unit 1)
 				)
@@
 		(on_board yes)
 		(dnp no)
-		(fields_autoplaced yes)
-		(property "Reference" "#PWR079"
+		(property "Reference" "#PWR081"
 			(at 83.82 29.21 0)
 			(effects
@@
 		)
 		(property "Value" "+3.3V_ISO"
-			(at 83.82 20.32 0)
+			(at 84.074 19.05 0)
 			(effects
 				(font
@@
 			(project "barn-blinds-controller"
 				(path "/aa90962a-81b9-423d-8acd-c4e83fa798bb/8f0cb6d8-027e-4edb-b8ea-04d7ddb83db1"
-					(reference "#PWR079")
-					(unit 1)
-				)
+					(reference "#PWR081")
+					(unit 1)
+				)

Commit message: V 1.2
Parts:
- added TP4: ASC Out, barn_shade_controller:TestPoint_Pad_D1.0mm_No_SolderMask, symbol Connector:TestPoint
Connections:
- net GPIO14 renamed ACS723
- net ACS723: now also TP4.1
- net GPIO15 renamed TMP235
Changed lines of the file:
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@@
+		(color 0 0 0 0)
+	)
+	(junction
+		(at 102.87 43.18)
+		(diameter 0)
 		(color 0 0 0 0)
 	)
@@
 	(no_connect
 		(at 71.12 85.09)
+	)
+	(wire
+		(pts
+			(xy 110.49 53.34) (xy 110.49 50.8)
+		)
+		(stroke
+			(width 0)
+			(type default)
+		)
 	)
 	(wire
@@
 	(wire
 		(pts
-			(xy 110.49 43.18) (xy 93.98 43.18)
+			(xy 110.49 43.18) (xy 102.87 43.18)
 		)
 		(stroke
@@
 	(wire
 		(pts
-			(xy 83.82 25.4) (xy 83.82 29.21)
+			(xy 102.87 43.18) (xy 93.98 43.18)
 		)
 		(stroke
@@
 	(wire
 		(pts
-			(xy 99.06 85.09) (xy 91.44 85.09)
+			(xy 83.82 25.4) (xy 83.82 29.21)
 		)
 		(stroke
@@
 	(wire
 		(pts
-			(xy 97.79 50.8) (xy 93.98 50.8)
+			(xy 99.06 85.09) (xy 91.44 85.09)
 		)
 		(stroke
@@
 	(wire
 		(pts
-			(xy 116.84 43.18) (xy 110.49 43.18)
+			(xy 97.79 50.8) (xy 93.98 50.8)
 		)
 		(stroke
@@
 		)
 	)
-	(hierarchical_label "GPIO15"
+	(wire
+		(pts
+			(xy 116.84 43.18) (xy 110.49 43.18)
+		)
+		(stroke
+			(width 0)
+			(type default)
+		)
+	)
+	(hierarchical_label "TMP235"
 		(shape input)
 		(at 71.12 90.17 180)
@@
 		)
 	)
-	(hierarchical_label "GPIO14"
+	(hierarchical_label "ACS723"
 		(shape input)
 		(at 116.84 43.18 0)
@@
 	(symbol
 		(lib_id "power:GND")
-		(at 110.49 50.8 0)
+		(at 110.49 53.34 0)
 		(unit 1)
 		(exclude_from_sim no)
@@
 		(fields_autoplaced yes)
 		(property "Reference" "#PWR087"
-			(at 110.49 57.15 0)
+			(at 110.49 59.69 0)
 			(effects
 				(font
@@
 		)
 		(property "Value" "GND_ISO"
-			(at 110.49 55.88 0)
+			(at 110.49 58.42 0)
 			(effects
 				(font
@@
 		)
 		(property "Footprint" ""
-			(at 110.49 50.8 0)
+			(at 110.49 53.34 0)
 			(effects
 				(font
@@
 		)
 		(property "Datasheet" ""
-			(at 110.49 50.8 0)
+			(at 110.49 53.34 0)
 			(effects
 				(font
@@
 		)
 		(property "Description" "Power symbol creates a global label with name \"GND\" , ground"
-			(at 110.49 50.8 0)
+			(at 110.49 53.34 0)
 			(effects
 				(font
@@
 					(unit 1)
 				)
+			)
+		)
+	)
+	(symbol
+		(lib_id "Connector:TestPoint")
+		(at 102.87 43.18 0)
+		(unit 1)
+		(exclude_from_sim no)
+		(in_bom yes)
+		(on_board yes)
+		(dnp no)
+		(fields_autoplaced yes)
+		(property "Reference" "TP4"
+			(at 105.41 38.6079 0)
+			(effects
+				(font
+					(size 1.27 1.27)
+				)
+				(justify left)
+			)
+		)
+		(property "Value" "ASC Out"
+			(at 105.41 41.1479 0)
+			(effects
+				(font
+					(size 1.27 1.27)
+				)
+				(justify left)
+			)
+		)
+		(property "Footprint" "barn_shade_controller:TestPoint_Pad_D1.0mm_No_SolderMask"
+			(at 107.95 43.18 0)
+			(effects
+				(font
+					(size 1.27 1.27)
+				)
+				(hide yes)
+			)
+		)
+		(property "Datasheet" "~"
+			(at 107.95 43.18 0)
+			(effects
+				(font
+					(size 1.27 1.27)
+				)
+				(hide yes)
+			)
+		)
+		(property "Description" "test point"
+			(at 102.87 43.18 0)
+			(effects
+				(font
+					(size 1.27 1.27)
+				)
+				(hide yes)
+			)
+		)
+		(pin "1"
+		)
+		(instances
+			(project "barn-blinds-controller"
+				(path "/aa90962a-81b9-423d-8acd-c4e83fa798bb/8f0cb6d8-027e-4edb-b8ea-04d7ddb83db1"
+					(reference "TP4")
+					(unit 1)
+				)
