File: sensors.kicad_sch (KiCad schematic)
At the start: 7 parts, among them U10 TMP235, U11 ACS723xLCTR-05AB

Commit message: Updating routing with new terminal block
Parts:
- TP7: renamed from TP4; footprint barn_shade_controller:TestPoint_Pad_D1.0mm_No_SolderMask -> TestPoint:TestPoint_Pad_D1.0mm

Commit message: Update annotations, fixed font sizes.
Parts:
- renumbered C_ACS1 to C18, C_ACS2 to C19, C_FILT1 to C20, C_TMP1 to C21
Changed lines of the file:
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@@
 		(dnp no)
 		(fields_autoplaced yes)
-		(property "Reference" "C_ACS2"
+		(property "Reference" "C19"
 			(at 114.3 45.7199 0)
 			(show_name no)
@@
 			(project "barn-blinds-controller"
 				(path "/aa90962a-81b9-423d-8acd-c4e83fa798bb/8f0cb6d8-027e-4edb-b8ea-04d7ddb83db1"
-					(reference "C_ACS2")
+					(reference "C19")
 					(unit 1)
 				)
@@
 		(dnp no)
 		(fields_autoplaced yes)
-		(property "Reference" "#PWR085"
+		(property "Reference" "#PWR087"
 			(at 97.79 29.21 0)
 			(hide yes)
@@
 			(project "barn-blinds-controller"
 				(path "/aa90962a-81b9-423d-8acd-c4e83fa798bb/8f0cb6d8-027e-4edb-b8ea-04d7ddb83db1"
-					(reference "#PWR085")
+					(reference "#PWR087")
 					(unit 1)
 				)
@@
 		(dnp no)
 		(fields_autoplaced yes)
-		(property "Reference" "C_ACS1"
+		(property "Reference" "C18"
 			(at 87.63 21.59 90)
 			(show_name no)
@@
 			(project "barn-blinds-controller"
 				(path "/aa90962a-81b9-423d-8acd-c4e83fa798bb/8f0cb6d8-027e-4edb-b8ea-04d7ddb83db1"
-					(reference "C_ACS1")
+					(reference "C18")
 					(unit 1)
 				)
@@
 		(dnp no)
 		(fields_autoplaced yes)
-		(property "Reference" "#PWR087"
+		(property "Reference" "#PWR089"
 			(at 99.06 99.06 0)
 			(hide yes)
@@
 			(project "barn-blinds-controller"
 				(path "/aa90962a-81b9-423d-8acd-c4e83fa798bb/8f0cb6d8-027e-4edb-b8ea-04d7ddb83db1"
-					(reference "#PWR087")
+					(reference "#PWR089")
 					(unit 1)
 				)
@@
 		(dnp no)
 		(fields_autoplaced yes)
-		(property "Reference" "#PWR086"
+		(property "Reference" "#PWR088"
 			(at 97.79 64.77 0)
 			(hide yes)
@@
 			(project "barn-blinds-controller"
 				(path "/aa90962a-81b9-423d-8acd-c4e83fa798bb/8f0cb6d8-027e-4edb-b8ea-04d7ddb83db1"
-					(reference "#PWR086")
+					(reference "#PWR088")
 					(unit 1)
 				)
@@
 		(dnp no)
 		(fields_autoplaced yes)
-		(property "Reference" "#PWR081"
+		(property "Reference" "#PWR083"
 			(at 77.47 43.18 0)
 			(hide yes)
@@
 			(project "barn-blinds-controller"
 				(path "/aa90962a-81b9-423d-8acd-c4e83fa798bb/8f0cb6d8-027e-4edb-b8ea-04d7ddb83db1"
-					(reference "#PWR081")
+					(reference "#PWR083")
 					(unit 1)
 				)
@@
 		(dnp no)
 		(fields_autoplaced yes)
-		(property "Reference" "#PWR089"
+		(property "Reference" "#PWR091"
 			(at 110.49 59.69 0)
 			(hide yes)
@@
 			(project "barn-blinds-controller"
 				(path "/aa90962a-81b9-423d-8acd-c4e83fa798bb/8f0cb6d8-027e-4edb-b8ea-04d7ddb83db1"
-					(reference "#PWR089")
+					(reference "#PWR091")
 					(unit 1)
 				)
@@
 		(dnp no)
 		(fields_autoplaced yes)
-		(property "Reference" "#PWR080"
+		(property "Reference" "#PWR082"
 			(at 64.77 87.63 0)
 			(hide yes)
@@
 			(project "barn-blinds-controller"
 				(path "/aa90962a-81b9-423d-8acd-c4e83fa798bb/8f0cb6d8-027e-4edb-b8ea-04d7ddb83db1"
-					(reference "#PWR080")
+					(reference "#PWR082")
 					(unit 1)
 				)
@@
 		(dnp no)
 		(fields_autoplaced yes)
-		(property "Reference" "#PWR088"
+		(property "Reference" "#PWR090"
 			(at 100.33 85.09 0)
 			(hide yes)
@@
 			(project "barn-blinds-controller"
 				(path "/aa90962a-81b9-423d-8acd-c4e83fa798bb/8f0cb6d8-027e-4edb-b8ea-04d7ddb83db1"
-					(reference "#PWR088")
+					(reference "#PWR090")
 					(unit 1)
 				)
@@
 		(dnp no)
 		(fields_autoplaced yes)
-		(property "Reference" "#PWR082"
+		(property "Reference" "#PWR084"
 			(at 77.47 50.8 0)
 			(hide yes)
@@
 			(project "barn-blinds-controller"
 				(path "/aa90962a-81b9-423d-8acd-c4e83fa798bb/8f0cb6d8-027e-4edb-b8ea-04d7ddb83db1"
-					(reference "#PWR082")
+					(reference "#PWR084")
 					(unit 1)
 				)
@@
 		(dnp no)
 		(fields_autoplaced yes)
-		(property "Reference" "#PWR084"
+		(property "Reference" "#PWR086"
 			(at 83.82 64.77 0)
 			(hide yes)
@@
 			(project "barn-blinds-controller"
 				(path "/aa90962a-81b9-423d-8acd-c4e83fa798bb/8f0cb6d8-027e-4edb-b8ea-04d7ddb83db1"
-					(reference "#PWR084")
+					(reference "#PWR086")
 					(unit 1)
 				)
@@
 		(dnp no)
 		(fields_autoplaced yes)
-		(property "Reference" "C_FILT1"
+		(property "Reference" "C20"
 			(at 101.6 53.3399 0)
 			(show_name no)
@@
 			(project "barn-blinds-controller"
 				(path "/aa90962a-81b9-423d-8acd-c4e83fa798bb/8f0cb6d8-027e-4edb-b8ea-04d7ddb83db1"
-					(reference "C_FILT1")
+					(reference "C20")
 					(unit 1)
 				)
@@
 		(dnp no)
 		(fields_autoplaced yes)
-		(property "Reference" "C_TMP1"
+		(property "Reference" "C21"
 			(at 102.87 87.6299 0)
 			(show_name no)
@@
 			(project "barn-blinds-controller"
 				(path "/aa90962a-81b9-423d-8acd-c4e83fa798bb/8f0cb6d8-027e-4edb-b8ea-04d7ddb83db1"
-					(reference "C_TMP1")
+					(reference "C21")
 					(unit 1)
 				)
@@
 		(in_pos_files yes)
 		(dnp no)
-		(property "Reference" "#PWR083"
+		(property "Reference" "#PWR085"
 			(at 83.82 29.21 0)
 			(hide yes)
@@
 			(project "barn-blinds-controller"
 				(path "/aa90962a-81b9-423d-8acd-c4e83fa798bb/8f0cb6d8-027e-4edb-b8ea-04d7ddb83db1"
-					(reference "#PWR083")
-					(unit 1)
-				)
+					(reference "#PWR085")
+					(unit 1)
+				)
