File: sensors.kicad_sch (KiCad schematic)
At the start: 7 parts, among them U10 TMP235, U11 ACS723xLCTR-05AB

Commit message: Pre-fab QA review fixes: switch input levels, power path, sensor spec, ESD
- R1-R8 switch series resistors 10k -> 1k: with only the ESP32 internal
  ~45k pull-up, 10k divided a closed switch to 0.6V vs the S3's 0.825V
  VIL limit — marginal. 1k gives ~0.1-0.23V worst case.
- U11 ACS723 -> ACS725LLCTR-05AB-T (C3684552): ACS723 needs 4.5-5.5V but
  ran at 3.3V (out of spec). ACS725 is 3.3V-native, same SOIC-8, rated
  to +150C. Firmware: sensitivity 264mV/A, formula (x-1.65)/0.264.
- D2 BAT54C (200mA) removed; replaced with D10/D11 SS34 (3A) diode-OR.
  The old diode carried the full ESP32 load permanently; WiFi TX bursts
  reach 350-500mA.
- U16 PRTR5V0U2X added on USB D+/D- (ESD protection at J2).
- D1 SS34 -> SS54 (5A, same SMA footprint) for multi-motor headroom.
- C10 bumped to 25V-rated 100uF 1210 (C2840614), same footprint.
- Filled all missing LCSC fields for JLCPCB assembly BOM.
- Docs: J4 pinout corrected to as-built; firmware bring-up checklist and
  RTS/DTR terminal gotcha added; CLAUDE.md placement guide for D10/D11/U16.

PCB placement of D10/D11/U16 + F8 sync still pending.

Co-Authored-By: Claude Fable 5 <noreply@anthropic.com>
Parts:
- U11: value ACS723xLCTR-05AB -> ACS725LLCTR-05AB-T; LCSC C2655492 -> C3684552
Changed lines of the file:
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@@
 			)
 		)
-		(property "Value" "ACS723xLCTR-05AB"
+		(property "Value" "ACS725LLCTR-05AB-T"
 			(at 85.9633 38.1 0)
 			(show_name no)
@@
 			)
 		)
-		(property "Datasheet" "http://www.allegromicro.com/~/media/Files/Datasheets/ACS723-Datasheet.ashx?la=en"
+		(property "Datasheet" "https://www.allegromicro.com/-/media/files/datasheets/acs725-datasheet.pdf"
 			(at 83.82 48.26 0)
 			(hide yes)
@@
 			)
 		)
-		(property "LCSC" "C2655492"
+		(property "LCSC" "C3684552"
 			(at 83.82 48.26 0)
 			(hide yes)

Commit message: Rev 1.3 PCB sync + second QA pass: BOM fixes, TVS decoupling, ERC cleanup
PCB (done in KiCad, verified here):
- F8 sync applied: D2 removed; D10/D11 (SS34 SMA) and U16 (PRTR5V0U2X SOT-143)
  placed and routed; R1-R8 -> 1k, D1 -> SS54, C10 -> 25V, U11 -> ACS725 updated
  in place. Footprint-level diff confirms exactly the intended delta, nothing
  else moved. DRC 0 errors / 0 unconnected pads.

Schematic fixes from the second QA pass:
- R1-R8 had NO LCSC part number (value change had landed, part number never
  did) - they would have come back unpopulated, silently killing the switch
  inputs. Set to C14676, matching R14's existing 1K 0603 so it consolidates to
  one BOM line. NOTE: todo.md originally specified C21190 - see the discrepancy
  note there and confirm before ordering.
- TP1-TP7 set in_bom no / in_pos_files no (were 7 junk lines in the JLCPCB BOM).
- Removed 4 orphan dangling wire stubs in switch_inputs.kicad_sch.
- Converted the orphan STBY hierarchical label in motor_drivers.kicad_sch to a
  global label rather than deleting it: its wire actually carried U9 pin 19, so
  deleting dropped U9.19 off the STBY net. Converting keeps the connection and
  clears the ERC hier_label_mismatch.
- Added C40-C43 (100nF 0402, C1525) for U12-U15 VCC decoupling. The switch-input
  TVS devices currently have their nearest +3.3V_ISO bypass 18-23mm away; a
  PRTR5V0U2X shunts ESD into VCC and needs somewhere local to dump it. Still
  need PCB placement - put each within ~2mm of its device's pin 4.

Every schematic edit was validated by diffing the exported netlist before and
after; connectivity is unchanged apart from the four intended new caps.
ERC errors: 10 -> 5 (remaining are 4x missing PWR_FLAG and one J2-GND/U1-(-Vout)
both-power-output pair that is correct by design).

Added barn-blinds-controller.kicad_dru: isolation-barrier audit rule. The board
has no dedicated ISO/MOTOR gap - minimum copper spacing between domains is
0.20mm, the global default. Rev 1.2 measured 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
Parts:
- TP7: now left out of the parts list
Changed lines of the file:
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@@
 		(body_style 1)
 		(exclude_from_sim no)
-		(in_bom yes)
+		(in_bom no)
 		(on_board yes)
-		(in_pos_files yes)
+		(in_pos_files no)
 		(dnp no)
 		(fields_autoplaced yes)
