File: barn-blinds-controller.kicad_sch (KiCad schematic)
At the start: 4 parts

Commit message: Rev 1.3 updates
Other:
- added sheet Switch Inputs (switch_inputs.kicad_sch)
Changed lines of the file:
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@@
+		)
+	)
+	(sheet
+		(at 179.8319 111.0)
+		(size 22.9466 20.0)
+		(exclude_from_sim no)
+		(in_bom yes)
+		(on_board yes)
+		(dnp no)
+		(fields_autoplaced yes)
+		(stroke
+			(width 0.1524)
+			(type solid)
+		)
+		(fill
+			(color 0 0 0 0.0000)
+		)
+		(property "Sheetname" "Switch Inputs"
+			(at 179.8319 110.2884 0)
+			(effects
+				(font
+					(size 1.27 1.27)
+				)
+				(justify left bottom)
+			)
+		)
+		(property "Sheetfile" "switch_inputs.kicad_sch"
+			(at 179.8319 131.584 0)
+			(effects
+				(font
+					(size 1.27 1.27)
+				)
+				(justify left top)
+			)
+		)
+		(instances
+			(project "barn-blinds-controller"
+				(path "/aa90962a-81b9-423d-8acd-c4e83fa798bb"
+					(page "9")
+				)
+			)
 		)
 	)
