File: motor_outputs.kicad_sch (KiCad schematic)
At the start: 9 parts, among them J4 Phoenix Contact 1786918

Commit message: Added RTS/DTS programing via UART circuitry, added LED control circuitry.
Parts:
- J4: footprint barn_shade_controller:Phoenix Contact 1786918 -> barn_shade_controller:1786918
Changed lines of the file:
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@@
 			)
 		)
-		(property "Footprint" "barn_shade_controller:Phoenix Contact 1786918"
+		(property "Footprint" "barn_shade_controller:1786918"
 			(at 160.02 164.77 0)
 			(hide yes)

Commit message: Update annotations, fixed font sizes.
Parts:
- renumbered D8 to D7, D9 to D8, D7 to D9
Changed lines of the file:
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@@
 		(dnp no)
 		(fields_autoplaced yes)
-		(property "Reference" "D7"
+		(property "Reference" "D9"
 			(at 76.2 125.7299 0)
 			(show_name no)
@@
 			(project "barn-blinds-controller"
 				(path "/aa90962a-81b9-423d-8acd-c4e83fa798bb/4857807b-67c7-42cb-aab6-84b757102806"
-					(reference "D7")
+					(reference "D9")
 					(unit 1)
 				)
@@
 		(dnp no)
 		(fields_autoplaced yes)
-		(property "Reference" "D8"
+		(property "Reference" "D7"
 			(at 78.74 76.1999 0)
 			(show_name no)
@@
 			(project "barn-blinds-controller"
 				(path "/aa90962a-81b9-423d-8acd-c4e83fa798bb/4857807b-67c7-42cb-aab6-84b757102806"
-					(reference "D8")
+					(reference "D7")
 					(unit 1)
 				)
@@
 		(dnp no)
 		(fields_autoplaced yes)
-		(property "Reference" "D9"
+		(property "Reference" "D8"
 			(at 80.01 101.5999 0)
 			(show_name no)
@@
 			(project "barn-blinds-controller"
 				(path "/aa90962a-81b9-423d-8acd-c4e83fa798bb/4857807b-67c7-42cb-aab6-84b757102806"
-					(reference "D9")
+					(reference "D8")
 					(unit 1)
 				)
