File: motor_outputs.kicad_sch (KiCad schematic)
At the start: 9 parts, among them J4 Phoenix Contact 1786918

Commit message: Rev 1.3 fab-ready: PICK UP HERE items closed, JLCPCB production files generated
PCB (verified via DRC/ERC/netlist diff, not just eyeballed):
- Placed C40-C43 within ~1.8-2.6mm of each PRTR5V0U2X VCC pin (U12-U15).
- Widened +5V_OR to 0.5mm and USB_VBUS to 0.4mm.
- Moved U16 closer to J2 (center-to-center 6.1mm -> 4.0mm). Still on B.Cu
  vs J2's F.Cu, so the D+/D- path still crosses layers via a short stub -
  accepted trade-off for a Full-Speed, occasional-use flashing port.
- Fixed D10/D11 silkscreen reference overlap.
- Added LCSC to J2 (C397452, Micro-USB) and J4 (C6652293 - pre-purchased
  JLCPCB inventory part; number is still required for JLCPCB to place it).

DRC: 0 unconnected pads, 0 real errors. Remaining flagged items are all
accepted: 21 isolation-barrier warnings (all >=0.20mm, same floor as Rev 1.2)
and 5 hole_clearance exclusions on J2's own NPTH-vs-pad geometry (footprint-
inherent, not routing-fixable - confirmed the new one is capped by the same
0.20mm pad edge as the pre-existing accepted ones, not by trace width).

ERC steady at 5 benign errors (4x missing PWR_FLAG, 1x J2-GND/U1-(-Vout)
both-power-output by design).

Docs:
- Fixed stale "U7 DCDC DNP" note in jlcpcb-export-steps.md - that referred
  to a pre-renumbering designator. Today U1 is the Heniper DC-DC and U7 is
  a real, actively-used AMS1117-3.3 feeding +3.3V_MOTOR (U4-U6, U8-U9 logic
  supply) that must NOT be DNP'd.
- Documented U1's actual situation instead: DCDC_HYBRID_SLC03_TEC2 is a
  shared THT footprint across three vendor DC-DC modules (Mean Well/Traco/
  Heniper), silkscreened per-hole M/H/T. This run uses the Heniper
  (C20622657, JLCPCB inventory). Same-numbered pads share nets regardless
  of vendor so there's no electrical risk, but BOM/CPL only carry one
  position+rotation for the whole footprint - added a note that the JLCPCB
  assembly order needs an explicit remark to populate only the H holes.
- Updated CLAUDE.md PICK UP HERE and vsp-wsc4-todo.md to reflect fab-ready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
Parts:
- J4: LCSC (none) -> C6652293
Changed lines of the file:
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@@
+			)
+		)
+		(property "LCSC" "C6652293"
+			(at 140.97 69.85 0)
+			(hide yes)
+			(show_name no)
+			(do_not_autoplace no)
+			(effects
+				(font
+					(size 1.27 1.27)
+				)
 			)
 		)
