File: motor_drivers.kicad_sch (KiCad schematic)
At the start: 24 parts, among them Q2 2N7002, U7 AMS1117-3.3, U8 TB6612FNG, U9 TB6612FNG

Commit message: Pre-fab QA review fixes: switch input levels, power path, sensor spec, ESD
- R1-R8 switch series resistors 10k -> 1k: with only the ESP32 internal
  ~45k pull-up, 10k divided a closed switch to 0.6V vs the S3's 0.825V
  VIL limit — marginal. 1k gives ~0.1-0.23V worst case.
- U11 ACS723 -> ACS725LLCTR-05AB-T (C3684552): ACS723 needs 4.5-5.5V but
  ran at 3.3V (out of spec). ACS725 is 3.3V-native, same SOIC-8, rated
  to +150C. Firmware: sensitivity 264mV/A, formula (x-1.65)/0.264.
- D2 BAT54C (200mA) removed; replaced with D10/D11 SS34 (3A) diode-OR.
  The old diode carried the full ESP32 load permanently; WiFi TX bursts
  reach 350-500mA.
- U16 PRTR5V0U2X added on USB D+/D- (ESD protection at J2).
- D1 SS34 -> SS54 (5A, same SMA footprint) for multi-motor headroom.
- C10 bumped to 25V-rated 100uF 1210 (C2840614), same footprint.
- Filled all missing LCSC fields for JLCPCB assembly BOM.
- Docs: J4 pinout corrected to as-built; firmware bring-up checklist and
  RTS/DTR terminal gotcha added; CLAUDE.md placement guide for D10/D11/U16.

PCB placement of D10/D11/U16 + F8 sync still pending.

Co-Authored-By: Claude Fable 5 <noreply@anthropic.com>
Parts:
- Q2: LCSC (none) -> C8545
Changed lines of the file:
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@@
+			)
+		)
+		(property "LCSC" "C8545"
+			(at 198.12 69.85 0)
+			(hide yes)
+			(show_name no)
+			(do_not_autoplace no)
+			(effects
+				(font
+					(size 1.27 1.27)
+				)
 			)
 		)
