File: motor_drivers.kicad_sch (KiCad schematic)
At the start: 24 parts, among them Q2 2N7002, U7 AMS1117-3.3, U8 TB6612FNG, U9 TB6612FNG

Commit message: Rev 1.3 PCB sync + second QA pass: BOM fixes, TVS decoupling, ERC cleanup
PCB (done in KiCad, verified here):
- F8 sync applied: D2 removed; D10/D11 (SS34 SMA) and U16 (PRTR5V0U2X SOT-143)
  placed and routed; R1-R8 -> 1k, D1 -> SS54, C10 -> 25V, U11 -> ACS725 updated
  in place. Footprint-level diff confirms exactly the intended delta, nothing
  else moved. DRC 0 errors / 0 unconnected pads.

Schematic fixes from the second QA pass:
- R1-R8 had NO LCSC part number (value change had landed, part number never
  did) - they would have come back unpopulated, silently killing the switch
  inputs. Set to C14676, matching R14's existing 1K 0603 so it consolidates to
  one BOM line. NOTE: todo.md originally specified C21190 - see the discrepancy
  note there and confirm before ordering.
- TP1-TP7 set in_bom no / in_pos_files no (were 7 junk lines in the JLCPCB BOM).
- Removed 4 orphan dangling wire stubs in switch_inputs.kicad_sch.
- Converted the orphan STBY hierarchical label in motor_drivers.kicad_sch to a
  global label rather than deleting it: its wire actually carried U9 pin 19, so
  deleting dropped U9.19 off the STBY net. Converting keeps the connection and
  clears the ERC hier_label_mismatch.
- Added C40-C43 (100nF 0402, C1525) for U12-U15 VCC decoupling. The switch-input
  TVS devices currently have their nearest +3.3V_ISO bypass 18-23mm away; a
  PRTR5V0U2X shunts ESD into VCC and needs somewhere local to dump it. Still
  need PCB placement - put each within ~2mm of its device's pin 4.

Every schematic edit was validated by diffing the exported netlist before and
after; connectivity is unchanged apart from the four intended new caps.
ERC errors: 10 -> 5 (remaining are 4x missing PWR_FLAG and one J2-GND/U1-(-Vout)
both-power-output pair that is correct by design).

Added barn-blinds-controller.kicad_dru: isolation-barrier audit rule. The board
has no dedicated ISO/MOTOR gap - minimum copper spacing between domains is
0.20mm, the global default. Rev 1.2 measured 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
Parts:
- TP6: now left out of the parts list
Changed lines of the file:
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@@
 		)
 	)
-	(hierarchical_label "STBY"
-		(shape input)
+	(global_label "STBY"
+		(shape bidirectional)
 		(at 86.36 114.3 180)
+		(fields_autoplaced yes)
 		(effects
 			(font
@@
 			(justify right)
 		)
+		(property "Intersheetrefs" "${INTERSHEET_REFS}"
+			(at 86.36 114.3 180)
+			(hide yes)
+			(show_name no)
+			(do_not_autoplace no)
+			(effects
+				(font
+					(size 1.27 1.27)
+				)
+				(justify right)
+			)
+		)
 	)
 	(symbol
@@
 		(body_style 1)
 		(exclude_from_sim no)
-		(in_bom yes)
+		(in_bom no)
 		(on_board yes)
-		(in_pos_files yes)
+		(in_pos_files no)
 		(dnp no)
 		(fields_autoplaced yes)
