File: switch_inputs.kicad_sch (KiCad schematic)
At the start: 24 parts, among them U12 PRTR5V0U2X, U13 PRTR5V0U2X, U14 PRTR5V0U2X, U15 PRTR5V0U2X

Commit message: Stock-driven part swaps (C10, U12-U16) + J3 DNP after BOM audit
C10 (isolated 5V_ISO bulk cap): 100uF 25V (C2840614) was out of stock at
JLCPCB. Swapped to 100uF 16V (C7432790, HGC1210R5107M160NSVK) - same 1210
footprint, no PCB rework. 16V chosen over 10V/6.3V alternatives to keep
DC-bias derating low on the ~5V rail (unregulated B1205S-3WR2L output).

U12-U16 (PRTR5V0U2X ESD protection): C12333 was out of stock. Swapped to
C5158049 (UMW/Youtai) - same SOT-143 footprint, no PCB rework. Checked
four other "PRTR5V0U2X"-labeled LCSC listings before picking this one -
they were mismatched (unidirectional, or 14-25V standoff instead of ~5V)
despite sharing the part name; C5158049 actually matches the real
bidirectional/0.35pF/5V-7.2V spec.

Both changes verified via netlist diff (only Value/LCSC fields changed,
zero connectivity impact) and ERC (still 5 known-benign errors).

Auditing the regenerated JLCPCB assembly-order BOM turned up a separate,
pre-existing bug: J3's LCSC (C492404) is a 5-pin header (PZ254V-11-05P),
mismatched against its 7-pin footprint - a leftover from before J3 grew
from 5->7 pins for the RTS/DTR rework, where the LCSC field (and a stale
"01x05" Description) never got updated. JLCPCB's assembly matcher didn't
flag the mismatch, it silently auto-substituted a different 5-pin part.
A real 7-pin replacement isn't in stock either, and J3 is only a backup
UART flashing path (native USB on GPIO19/20 is primary) - not worth
chasing for this run, so J3 is now marked DNP. Fixed the stale "01x05"
Description text to "01x07" so the record is correct if it's ever
un-DNP'd (LCSC still needs a real 7-pin part first if that happens).

PCB: C10/U12-U16 changes synced via F8. J3's new DNP flag still needs an
F8 sync (done after the schematic edit, not yet reflected on the board).

Updated CLAUDE.md PICK UP HERE and vsp-wsc4-todo.md with full detail.
VSP-WSC-4_1.3 production files predate all three changes - needs a
Fabrication Toolkit re-run before ordering.

Co-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
Parts:
- U12, U13, U14, U15: LCSC C12333 -> C5158049
Changed lines of the file:
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@@
 			)
 		)
-		(property "LCSC" "C12333"
+		(property "LCSC" "C5158049"
 			(at 135.89 33.02 0)
 			(hide yes)
@@
 			)
 		)
-		(property "LCSC" "C12333"
+		(property "LCSC" "C5158049"
 			(at 133.35 152.4 0)
 			(hide yes)
@@
 			)
 		)
-		(property "LCSC" "C12333"
+		(property "LCSC" "C5158049"
 			(at 135.89 76.2 0)
 			(hide yes)
@@
 			)
 		)
-		(property "LCSC" "C12333"
+		(property "LCSC" "C5158049"
 			(at 133.35 111.76 0)
 			(hide yes)
